File: four_probe.sch (KiCad schematic (older format))
At the start: 15 parts

Commit message: update
Parts:
- removed J?: V_test, symbol Conn_01x02
- removed J?: V_TRANS, symbol Conn_01x01
- removed U?: OPA4340EA, symbol OPA4340EA
- added C50, C84, C? (x2): 1 nF, symbol C
- added Q1, Q2: Q_PNP_BCE, symbol Q_PNP_BCE
- added R34, R41, R? (x2): 430, symbol R
- added R? (x2), R_g: R, symbol R
- added R? (x2): 1K, symbol R
- added U15: AD620, symbol AD620
- added U16, U19, U? (x2): Jelly Bean, TO_SOT_Packages_SMD:SOT-23-5, symbol LM321
Connections:
- net GND: now also U15.4 (Vs-), U16.2 (V-), U19.2 (V-), U?.2 (V-), U?.2 (V-)
- net GNDREF: now also C50.1, C84.1, U19.1 (+), U?.1 (+)
- net VCC: now also U15.7 (Vs+), U16.5 (V+), U19.5 (V+), U?.5 (V+), U?.5 (V+)
- net at C?.1, R_f.1: now also R?.2, U19.4
- net at C?.2, J?.1 (Pin_1), R_f.2: now also U19.3 (-)
- net at J?.1 (Pin_1): now also U15.3 (+)
- net at J?.1 (Pin_1): now also U15.2 (-)
- new net: R_g.2, U15.1 (Rg)
- new net: U15.5 (Ref), U?.3 (-), U?.4
- new net: R?.2, U15.6
- new net: R_g.1, U15.8 (Rg)
- new net: Q1.3 (E), R?.1
- new net: Q2.3 (E), R?.1
- new net: Q2.1 (B), R?.2
- new net: Q2.2 (C), R41.2
- new net: C84.2, R41.1, U16.1 (+)
- new net: Q1.1 (B), R?.2
- new net: Q1.2 (C), R34.2
- new net: C50.2, R34.1, U?.1 (+)
- new net: C?.2, R?.1, U?.3 (-)
- new net: C?.2, R?.1, U16.3 (-)
- new net ADC_current: C?.1, R?.2, U16.4
- new net ADC_voltage: C?.1, R?.2, U?.4
- new net PWM1: R?.1, R?.1
Other:
- note added: "Current Sense"
- note added: "Four Probe v_0.2"
- note added: "Input Signal ( +VEXC, -VEXC)"
- note added: "Set gain for current"
- note added: "Set gain for voltage"
- note added: "Switch for +VEXC"
- note removed: "Current Sense\n"
- note removed: "Current_test = (GNDREF - V_TRANS) / R_f"
- note removed: "Four Probe Test Circuit"
- note removed: "Four Probes In Solution"
- note removed: "Input Signal"
- note removed: "R_test = V_test / Current_test"
- moved on the sheet: C?, J?, R?, R_f, R_limit

Commit message: update
Parts:
- C84: value 1 nF -> 1nF
- CF1, CF2: renamed from C?; value 1 nF -> 1nF
- CT1: renamed from C?; value C -> 1nF
- R_f: value R -> R47
- gave numbers to parts that had none: 6
Changed lines of the file:
@@
 P 3500 4250
 F 0 "R_f" V 3580 4250 50  0000 C CNN
-F 1 "R" V 3500 4250 50  0000 C CNN
+F 1 "R47" V 3500 4250 50  0000 C CNN
 F 2 "" V 3430 4250 50  0001 C CNN
 F 3 "" H 3500 4250 50  0001 C CNN
@@
 $EndComp
 $Comp
-L C C?
+L C CT1
 U 1 1 5AC56DCB
 P 3500 3950
-F 0 "C?" H 3525 4050 50  0000 L CNN
-F 1 "C" H 3525 3850 50  0000 L CNN
+F 0 "CT1" V 3450 3750 50  0000 L CNN
+F 1 "1nF" V 3450 4000 50  0000 L CNN
 F 2 "" H 3538 3800 50  0001 C CNN
 F 3 "" H 3500 3950 50  0001 C CNN
@@
 $EndComp
 $Comp
-L LM321 U?
+L LM321 U22B
 U 1 1 5ACC098A
 P 5300 3000
-F 0 "U?" H 5250 3000 50  0000 L CNN
+F 0 "U22B" H 5250 3000 50  0000 L CNN
 F 1 "Jelly Bean" H 5350 3150 50  0000 L CNN
 F 2 "TO_SOT_Packages_SMD:SOT-23-5" H 5300 3000 50  0001 C CNN
@@
 $EndComp
 $Comp
-L R R?
+L R RS1
 U 1 1 5ACC0CB0
 P 5850 2100
-F 0 "R?" V 5930 2100 50  0000 C CNN
+F 0 "RS1" V 5930 2100 50  0000 C CNN
 F 1 "430" V 5850 2100 50  0000 C CNN
 F 2 "" V 5780 2100 50  0001 C CNN
@@
 Text Notes 3400 2400 0    60   ~ 0
 Set gain for voltage
-Text Notes 3800 3850 0    60   ~ 0
+Text Notes 3950 4150 0    60   ~ 0
 Set gain for current
 $Comp
-L R R?
+L R RS2
 U 1 1 5ACC71CD
 P 4250 4750
-F 0 "R?" V 4330 4750 50  0000 C CNN
+F 0 "RS2" V 4330 4750 50  0000 C CNN
 F 1 "430" V 4250 4750 50  0000 C CNN
 F 2 "" V 4180 4750 50  0001 C CNN
@@
 Switch for +VEXC
 $Comp
-L LM321 U?
+L LM321 U10
 U 1 1 5ACCD490
 P 8150 2200
-F 0 "U?" H 8100 2200 50  0000 L CNN
+F 0 "U10" H 8100 2200 50  0000 L CNN
 F 1 "Jelly Bean" H 8200 2350 50  0000 L CNN
 F 2 "TO_SOT_Packages_SMD:SOT-23-5" H 8150 2200 50  0001 C CNN
@@
 $EndComp
 $Comp
-L R R?
+L R RF1
 U 1 1 5ACCE3E9
 P 8150 2900
-F 0 "R?" V 8230 2900 50  0000 C CNN
+F 0 "RF1" V 8230 2900 50  0000 C CNN
 F 1 "1K" V 8150 2900 50  0000 C CNN
 F 2 "" V 8080 2900 50  0001 C CNN
@@
 $EndComp
 $Comp
-L C C?
+L C CF1
 U 1 1 5ACCE814
 P 8150 3200
-F 0 "C?" V 8200 3050 50  0000 L CNN
-F 1 "1 nF" V 8300 3100 50  0000 L CNN
+F 0 "CF1" V 8200 3000 50  0000 L CNN
+F 1 "1nF" V 8200 3250 50  0000 L CNN
 F 2 "" H 8188 3050 50  0001 C CNN
 F 3 "" H 8150 3200 50  0001 C CNN
@@
 $EndComp
 $Comp
-L R R?
+L R RF2
 U 1 1 5ACD1549
 P 6400 5550
-F 0 "R?" V 6480 5550 50  0000 C CNN
+F 0 "RF2" V 6480 5550 50  0000 C CNN
 F 1 "1K" V 6400 5550 50  0000 C CNN
 F 2 "" V 6330 5550 50  0001 C CNN
@@
 P 5700 4900
 F 0 "C84" H 5725 5000 50  0000 L CNN
-F 1 "1 nF" H 5500 5000 50  0000 L CNN
+F 1 "1nF" H 5500 5000 50  0000 L CNN
 F 2 "" H 5738 4750 50  0001 C CNN
 F 3 "" H 5700 4900 50  0001 C CNN
@@
 	3400 4450 3550 4450
 Wire Wire Line
-	3200 3950 3200 4650
-Wire Wire Line
-	3800 3950 3800 4750
+	3200 3950 3200 4250
+Wire Wire Line
+	3200 4250 3200 4650
+Wire Wire Line
+	3800 3950 3800 4250
+Wire Wire Line
+	3800 4250 3800 4750
 Wire Wire Line
 	3200 4850 3050 4850
@@
 	4800 2900 4800 2950
 Wire Wire Line
-	5600 3600 5600 2400
+	5600 3600 5600 3000
+Wire Wire Line
+	5600 3000 5600 2400
 Wire Wire Line
 	5600 2400 5000 2400
@@
 	6000 2100 6300 2100
 Wire Notes Line
-	3900 3900 3900 4100
-Wire Notes Line
 	3900 4100 3500 4100
 Wire Wire Line
@@
 	6700 2100 6950 2100
 Wire Wire Line
-	7250 2100 7850 2100
-Wire Wire Line
-	7850 2300 7850 3200
-Wire Wire Line
-	8450 2200 8450 3200
+	7250 2100 7400 2100
+Wire Wire Line
+	7400 2100 7850 2100
+Wire Wire Line
+	7850 2300 7850 2900
+Wire Wire Line
+	7850 2900 7850 3200
+Wire Wire Line
+	8450 2200 8450 2900
+Wire Wire Line
+	8450 2900 8450 3200
 Wire Wire Line
 	7850 3200 8000 3200
@@
 	8450 2200 8850 2200
 Wire Wire Line
-	5550 4750 6100 4750
-Wire Wire Line
-	6100 4950 6100 5850
-Wire Wire Line
-	6700 4850 6700 5850
+	5550 4750 5700 4750
+Wire Wire Line
+	5700 4750 6100 4750
+Wire Wire Line
+	6100 4950 6100 5550
+Wire Wire Line
+	6100 5550 6100 5850
+Wire Wire Line
+	6700 4850 6700 5550
+Wire Wire Line
+	6700 5550 6700 5850
 Wire Wire Line
 	6100 5850 6250 5850
@@
 Connection ~ 5700 4750
 $Comp
-L C C?
+L C CF2
 U 1 1 5ACE0809
 P 6400 5850
-F 0 "C?" V 6450 5700 50  0000 L CNN
-F 1 "1 nF" V 6550 5750 50  0000 L CNN
+F 0 "CF2" V 6450 5650 50  0000 L CNN
+F 1 "1nF" V 6450 5950 50  0000 L CNN
 F 2 "" H 6438 5700 50  0001 C CNN
 F 3 "" H 6400 5850 50  0001 C CNN

Commit message: update
Parts:
- added U22B?: Jelly Bean, TO_SOT_Packages_SMD:SOT-23-5, symbol LM321
Connections:
- net GND: now also U22B?.2 (V-)
- net GNDREF: now also U22B?.3 (-), U22B?.4; no longer R?.1, R?.2
- net VCC: now also U22B?.5 (V+)
- new net: R?.1, R?.2, U22B?.1 (+)
Other:
- note added: "Four Probe v_0.3"
- note added: "Power Input"
- note removed: "Four Probe v_0.2"
- moved on the sheet: C50, C84, C?, CF1, CF2, CT1, J?, Q1, Q2, R34, R41, R?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
