File: v_0.4/four_probe.sch (KiCad schematic (older format))
At the start: 81 parts, among them U10 Jelly Bean, U15 AD620, U16 Jelly Bean, U19 Jelly Bean, U22B Jelly Bean, U22B? Jelly Bean

Commit message: update
Other:
- note added: "Four Probe v_0.4"
Changed lines of the file:
@@
 Wire Wire Line
 	2400 7950 2400 10150
-Text Notes 1000 8300 0    100  ~ 0
+Text Notes 2550 9950 0    100  ~ 0
 CURRENT SENSE
-Text Notes 8500 9600 0    100  ~ 0
+Text Notes 8850 9850 0    100  ~ 0
 CURRENT SENSE
 Text Notes 8950 2600 0    100  ~ 0
@@
 	9900 8100 10200 8100
 Connection ~ 10200 8100
+Text Notes 13200 9700 0    200  ~ 0
+Four Probe v_0.4
 $EndSCHEMATC

Commit message: update
Connections:
- net VCC: no longer R?.2
Other:
- note added: "Switch for -VEXC"
- moved on the sheet: C50, C84, C?, CF2, CF?, CT?, J?, R34, R41, R?, RF1, RF2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
