File: v_0.5/four_probe.sch (KiCad schematic (older format))
At the start: 77 parts, among them J1 Power_input, J12 Conn_01x03_Female, U1 LMC6482, U10 ADG704, U2 AD623, U3 LMC6482, U4 AD623, U5 LMC6484, U6 LMC6484, U7 ADG1212, U8 ADG704, U9 ADG704

Commit message: update
Other:
- note added: "PWM Inputs"
- note added: "Probes"
- note added: "Voltage Inputs"
- moved on the sheet: JP1, JPWM1, JVIN1
Changed lines of the file:
@@
 L Conn_01x04_Female JP1
 U 1 1 5AF5542B
-P 3400 5800
-F 0 "JP1" H 3400 6000 50  0000 C CNN
-F 1 "Conn_01x04_Female" H 3400 5500 50  0000 C CNN
-F 2 "" H 3400 5800 50  0001 C CNN
-F 3 "" H 3400 5800 50  0001 C CNN
-	1    3400 5800
+P 3500 5950
+F 0 "JP1" H 3500 6150 50  0000 C CNN
+F 1 "Conn_01x04_Female" H 3500 5650 50  0000 C CNN
+F 2 "" H 3500 5950 50  0001 C CNN
+F 3 "" H 3500 5950 50  0001 C CNN
+	1    3500 5950
 	1    0    0    -1
 $EndComp
@@
 Text GLabel 4400 5600 0    60   Input ~ 0
 P3
-Text GLabel 3200 6000 0    60   Input ~ 0
+Text GLabel 3300 6150 0    60   Input ~ 0
 PT4
-Text GLabel 3200 5900 0    60   Input ~ 0
+Text GLabel 3300 6050 0    60   Input ~ 0
 PT3
-Text GLabel 3200 5800 0    60   Input ~ 0
+Text GLabel 3300 5950 0    60   Input ~ 0
 PT2
-Text GLabel 3200 5700 0    60   Input ~ 0
+Text GLabel 3300 5850 0    60   Input ~ 0
 PT1
 Text GLabel 6200 5350 2    60   Input ~ 0
@@
 Text GLabel 13700 5400 0    60   Input ~ 0
 TIC
-Text GLabel 13700 5200 0    60   Input ~ 0
+Text GLabel 13300 5200 0    60   Input ~ 0
 TIA
-Text GLabel 13700 5300 0    60   Input ~ 0
+Text GLabel 13500 5300 0    60   Input ~ 0
 TIB
 $Comp
 L Conn_01x04_Female JVIN1
 U 1 1 5B018DB6
-P 4800 8500
-F 0 "JVIN1" H 4800 8700 50  0000 C CNN
-F 1 "Conn_01x04_Female" H 4800 8200 50  0000 C CNN
-F 2 "" H 4800 8500 50  0001 C CNN
-F 3 "" H 4800 8500 50  0001 C CNN
-	1    4800 8500
-	1    0    0    -1
-$EndComp
-Text GLabel 4600 8400 0    60   Input ~ 0
+P 1900 6950
+F 0 "JVIN1" H 1900 7150 50  0000 C CNN
+F 1 "Conn_01x04_Female" H 1900 6650 50  0000 C CNN
+F 2 "" H 1900 6950 50  0001 C CNN
+F 3 "" H 1900 6950 50  0001 C CNN
+	1    1900 6950
+	1    0    0    -1
+$EndComp
+Text GLabel 1700 6850 0    60   Input ~ 0
 VIN1
-Text GLabel 4600 8500 0    60   Input ~ 0
+Text GLabel 1700 6950 0    60   Input ~ 0
 VIN2
-Text GLabel 4600 8600 0    60   Input ~ 0
+Text GLabel 1700 7050 0    60   Input ~ 0
 VIN3
-Text GLabel 4600 8700 0    60   Input ~ 0
+Text GLabel 1700 7150 0    60   Input ~ 0
 VIN3
 Text GLabel 4000 9600 0    60   Input ~ 0
@@
 L Conn_01x02_Female JPWM1
 U 1 1 5B023455
-P 2400 8300
-F 0 "JPWM1" H 2400 8400 50  0000 C CNN
-F 1 "Conn_01x02_Female" H 2400 8100 50  0000 C CNN
-F 2 "" H 2400 8300 50  0001 C CNN
-F 3 "" H 2400 8300 50  0001 C CNN
-	1    2400 8300
-	1    0    0    -1
-$EndComp
-Text GLabel 2200 8300 0    60   Input ~ 0
+P 1950 7900
+F 0 "JPWM1" H 1950 8000 50  0000 C CNN
+F 1 "Conn_01x02_Female" H 1950 7700 50  0000 C CNN
+F 2 "" H 1950 7900 50  0001 C CNN
+F 3 "" H 1950 7900 50  0001 C CNN
+	1    1950 7900
+	1    0    0    -1
+$EndComp
+Text GLabel 1750 7900 0    60   Input ~ 0
 PWM1
-Text GLabel 2200 8400 0    60   Input ~ 0
+Text GLabel 1750 8000 0    60   Input ~ 0
 PWM2
 Wire Wire Line
@@
 	4500 6300 4400 6300
 Connection ~ 4500 6550
+Wire Wire Line
+	13300 5200 13700 5200
+Wire Wire Line
+	13500 5300 13700 5300
+Text Notes 1250 7650 0    98   ~ 0
+PWM Inputs
+Text Notes 1200 6550 0    98   ~ 0
+Voltage Inputs
+Text Notes 3050 5650 0    98   ~ 0
+Probes
 $EndSCHEMATC

Commit message: update
Parts:
- C1, C2, C3, C5, C50, C84, CF1, CF2, CF3, CF4, CF5, CF6, CG1, CG2, CT1, CT2, CT3, CT4, CU1, CU10, CU2, CU3, CU4, CU5, CU6, CU7, CU8, CU9: footprint (none) -> Capacitor_SMD:C_0603_1608Metric; symbol C -> four_probe-rescue:C
- J1, JRG4, JRL4, JRV12G1, JRV23G1: footprint (none) -> Connector_PinSocket_2.54mm:PinSocket_1x02_P2.54mm_Vertical; symbol Conn_01x02 -> four_probe-rescue:Conn_01x02
- J12, JTI1: footprint (none) -> Connector_PinSocket_2.54mm:PinSocket_1x03_P2.54mm_Vertical; symbol Conn_01x03_Female -> four_probe-rescue:Conn_01x03_Female
- JP1: footprint (none) -> Connector_PinSocket_2.54mm:PinSocket_2x02_P2.54mm_Vertical; symbol Conn_01x04_Female -> four_probe-rescue:Conn_01x04_Female
- JPWM1: footprint (none) -> Connector_PinSocket_2.54mm:PinSocket_1x02_P2.54mm_Vertical; symbol Conn_01x02_Female -> four_probe-rescue:Conn_01x02_Female
- JVIN1: footprint (none) -> Connector_PinSocket_2.54mm:PinSocket_1x04_P2.54mm_Vertical; symbol Conn_01x04_Female -> four_probe-rescue:Conn_01x04_Female
- R1, R2, R3, R34, R4, R41, R5, R6, RF1, RF2, RF3, RF4, RF5, RF6, RF7, RF8, RG1, RG2, RG3, RG4, RL1, RL2, RL3, RL4A1, RS1, RS2, RS3, RV12G1, RV23G1: footprint (none) -> Resistor_SMD:R_0603_1608Metric; symbol R -> four_probe-rescue:R
- U1, U3: symbol LMC6482 -> four_probe-rescue:LMC6482
- U10, U8, U9: symbol ADG704 -> adg704:ADG704
- U2, U4: footprint (none) -> Package_SO:SOIC-8_3.9x4.9mm_P1.27mm; symbol AD623 -> four_probe-rescue:AD623
- U5, U6: symbol LMC6484 -> four_probe-rescue:LMC6484
- U7: symbol ADG1212 -> adg1212:ADG1212
