File: v_0.6/four_probe.sch (KiCad schematic (older format))
At the start: 73 parts, among them J1 Conn_02x13_Counter_Clockwise, J2 RG, U1 LMC6482, U10 ADG704, U2 AD623, U3 LMC6482, U4 AD623, U5 LMC6484, U6 LMC6484, U7 DG421LE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

Commit message: update
Parts:
- J1: footprint Connector_Molex:Molex_Picoflex_90325-0026_2x13_P1.27mm_Vertical -> Connector_PinSocket_2.54mm:PinSocket_1x26_P2.54mm_Vertical
Connections:
- net PWM1-S: now also RS1.1, RS2.1, RS3.1
- net VIN3: no longer J1.6 (Pin_6)
- net VIN4: now also J1.6 (Pin_6)
Changed lines of the file:
@@
 VIN3
 Text GLabel 13150 2800 0    60   Input ~ 0
-VIN3
+VIN4
 Text GLabel 4000 9600 0    60   Input ~ 0
 VIN3
@@
 PWM2
 Wire Wire Line
-	7250 4900 7250 6650
-Wire Wire Line
-	7250 1200 7250 2950
+	7250 4900 7250 5800
+Wire Wire Line
+	7250 1200 7250 2100
 Wire Wire Line
 	4800 2300 5200 2300
@@
 	8500 2950 8650 2950
 Wire Wire Line
-	6000 2100 6950 2100
-Wire Wire Line
 	6300 2400 5700 2400
 Wire Wire Line
@@
 	11850 7450 11850 7550
 Wire Wire Line
-	13000 6300 13000 8050
-Wire Wire Line
-	12250 7150 12700 7150
+	13000 6300 13000 7150
 Wire Wire Line
 	6200 5350 6000 5350
@@
 Wire Wire Line
 	6000 1600 6100 1600
-Connection ~ 12250 7150
 Wire Wire Line
 	14800 6500 14800 7050
@@
 Wire Wire Line
 	9700 5000 10050 5000
-Connection ~ 6000 2100
 Connection ~ 6000 5800
 Wire Wire Line
@@
 F 0 "J1" H 13400 3717 50  0000 C CNN
 F 1 "Conn_02x13_Counter_Clockwise" V 13400 2900 50  0000 C CNN
-F 2 "Connector_Molex:Molex_Picoflex_90325-0026_2x13_P1.27mm_Vertical" H 13350 2900 50  0001 C CNN
+F 2 "Connector_PinSocket_2.54mm:PinSocket_1x26_P2.54mm_Vertical" H 13350 2900 50  0001 C CNN
 F 3 "~" H 13350 2900 50  0001 C CNN
 	1    13350 2900
@@
 	1    0    0    -1
 $EndComp
+Connection ~ 13000 7150
+Wire Wire Line
+	13000 7150 13000 8050
+Wire Wire Line
+	12700 7150 12250 7150
+Connection ~ 12250 7150
+Connection ~ 7250 5800
+Wire Wire Line
+	7250 5800 7250 6650
+Connection ~ 6000 2100
+Wire Wire Line
+	6000 2100 6950 2100
+Connection ~ 7250 2100
+Wire Wire Line
+	7250 2100 7250 2950
 $EndSCHEMATC
