File: v_0.6/four_probe.kicad_pcb (KiCad board)
At the start: 2 copper layers, 22.9 x 87.6 mm, 73 parts, among them J1 Conn_02x13_Counter_Clockwise, J2 RG, U1 LMC6482, U10 ADG704, U2 AD623, U3 LMC6482, U4 AD623, U5 LMC6484, U6 LMC6484, U7 DG421LE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

Commit message: update
Parts:
- J1: footprint Connector_Molex:Molex_Picoflex_90325-0026_2x13_P1.27mm_Vertical -> Connector_PinSocket_2.54mm:PinSocket_1x26_P2.54mm_Vertical
- moved CU1 87.7 mm to (23.2, 35.6)
- moved CU6 87.5 mm to (28.7, 21.6), turned to 180 degrees
- moved RG4 86.0 mm to (38.0, 52.5), turned to 90 degrees
- moved RG1 83.8 mm to (36.7, 72.3)
- moved RL2 78.2 mm to (28.6, 36.4), turned to 90 degrees
- moved RL4A1 77.3 mm to (27.6, 64.1), turned to 180 degrees
- moved CU4 71.8 mm to (20.3, 47.4), turned to 90 degrees
- moved RL3 70.2 mm to (31.4, 36.4), turned to 90 degrees
- moved RG3 69.7 mm to (41.3, 65.5)
- moved CT3 69.2 mm to (31.8, 46.9)
- moved CU7 68.5 mm to (20.2, 41.1), turned to 270 degrees
- moved RL1 67.1 mm to (26.4, 60.6)
- moved RG2 66.5 mm to (38.1, 62.6)
- moved R41 65.9 mm to (38.0, 84.7), turned to 270 degrees
- moved RF6 65.5 mm to (56.5, 77.1), turned to 270 degrees
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Connections:
- J1 pad 6: VIN3 -> VIN4
- RS1 pad 1: (no net) -> PWM1-S
- RS2 pad 1: (no net) -> PWM1-S
- RS3 pad 1: (no net) -> PWM1-S
- U9 pad 7: (no net) -> VIN4
Routing:
- net VIN1: track 0.00 -> 82.4 mm
- net VIN2: track 0.00 -> 70.6 mm
- net VIN3: track 0.00 -> 68.6 mm
- net VCC: track 0.00 -> 44.5 mm, vias 0 -> 1
- net GND: track 0.00 -> 32.9 mm, vias 0 -> 1
Other:
- board outline removed

Commit message: update
Parts:
- moved U8 103.7 mm to (100.5, -27.6), turned to 0 degrees
- moved U6 97.6 mm to (102.6, -11.8)
- moved U7 94.0 mm to (67.7, -8.76)
- moved U5 72.7 mm to (81.2, -19.6)
- moved U3 67.5 mm to (62.7, -22.9), turned to 0 degrees
- moved U10 65.0 mm to (36.7, -11.3), turned to 0 degrees
- moved U4 59.3 mm to (49.9, -9.02), turned to 0 degrees
- moved U2 54.1 mm to (46.7, -23.0)
- moved U9 50.9 mm to (14.7, -21.8), turned to 0 degrees
- moved U1 48.6 mm to (30.4, -21.7), turned to 0 degrees
Routing:
- net VCC: track 44.5 -> 232.9 mm, vias 1 -> 2
- net GND: track 32.9 -> 181.1 mm, vias 1 -> 4
- net VIN1: track 82.4 -> 0.00 mm
- net VIN2: track 70.6 -> 0.00 mm
- net VIN3: track 68.6 -> 1.20 mm
