File: v_0.7/four_probe.sch (KiCad schematic (older format))
At the start: 73 parts, among them J1 Conn_02x13_Counter_Clockwise, J2 RG, U1 LMC6482, U10 ADG704, U2 AD623, U3 LMC6482, U4 AD623, U5 LMC6484, U6 LMC6484, U7 DG421LE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

Commit message: update
Parts:
- added U?: ADG733BRU, Package_SO:TSSOP-20_4.4x6.5mm_P0.65mm, symbol Analog_Switch:ADG733BRU
- added U?: ADG1212, symbol adg1212:ADG1212
Changed lines of the file:
@@
 Wire Wire Line
 	7250 2100 7250 2950
+$Comp
+L Analog_Switch:ADG733BRU U?
+U 1 1 5CEFA9A2
+P -2100 450
+F 0 "U?" H -2100 692 50  0000 C CNN
+F 1 "ADG733BRU" H -2100 601 50  0000 C CNN
+F 2 "Package_SO:TSSOP-20_4.4x6.5mm_P0.65mm" H -2100 450 50  0001 C CNN
+F 3 "http://www.analog.com/media/en/technical-documentation/data-sheets/ADG733_734.pdf" H -2100 450 50  0001 C CNN
+	1    -2100 450
+	1    0    0    -1
+$EndComp
+$Comp
+L adg1212:ADG1212 U?
+U 1 1 5CEFAB82
+P -650 1300
+F 0 "U?" H -675 2087 60  0000 C CNN
+F 1 "ADG1212" H -675 1981 60  0000 C CNN
+F 2 "" H -650 1200 60  0001 C CNN
+F 3 "" H -650 1200 60  0001 C CNN
+	1    -650 1300
+	1    0    0    -1
+$EndComp
 $EndSCHEMATC

Commit message: update
Parts:
- removed U7: DG421LE, Package_SO:TSSOP-16_4.4x5mm_P0.65mm, symbol DG421LE:DG421LE
- removed U?: ADG733BRU, Package_SO:TSSOP-20_4.4x6.5mm_P0.65mm, symbol Analog_Switch:ADG733BRU
- removed U?: ADG1212, symbol adg1212:ADG1212
- added U11, U7: adg1211, digikey-footprints:TSSOP-16-1EP_W4.40mm, symbol adg1211:adg1211
- J1: symbol Connector_Generic:Conn_02x13_Counter_Clockwise -> four_probe-rescue:Conn_02x13_Counter_Clockwise-Connector_Generic
- J2: symbol Connector:Conn_01x02_Female -> four_probe-rescue:Conn_01x02_Female-Connector
Connections:
- net GND: now also U11.4 (VSS), U11.5 (GND), U7.4 (VSS), U7.5 (GND)
- net PWM1: now also U11.1 (IN1), U7.1 (IN1), U7.9 (IN3)
- net PWM2: now also U11.16 (IN2), U7.16 (IN2), U7.8 (IN4)
- removed net PWM1-D: R3.2, R41.2, R5.2
- removed net PWM1-S: RS1.1, RS2.1, RS3.1
- removed net PWM2-D: R34.2, R4.2, R6.2
- new net: RS1.1, U7.11 (S3), U7.6 (S4)
- new net: RS2.1, U11.14 (S2), U11.3 (S1)
- new net: R41.2, U11.2 (D1)
- new net: R34.2, U7.7 (D4)
- new net: R5.2, U7.10 (D3)
- new net: R6.2, U11.15 (D2)
- new net: RS3.1, U7.14 (S2), U7.3 (S1)
- new net: R4.2, U7.15 (D2)
- new net: R3.2, U7.2 (D1)
