File: v_0.7/four_probe.kicad_pcb (KiCad board)
At the start: 2 copper layers, 73 parts, among them J1 Conn_02x13_Counter_Clockwise, J2 RG, U1 LMC6482, U10 ADG704, U2 AD623, U3 LMC6482, U4 AD623, U5 LMC6484, U6 LMC6484, U7 DG421LE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

Commit message: update
Parts:
- added U11: adg1211, digikey-footprints:TSSOP-16-1EP_W4.40mm, F.Cu at (36.0, -27.9)
- U7: value DG421LE -> adg1211; footprint Package_SO:TSSOP-16_4.4x5mm_P0.65mm -> digikey-footprints:TSSOP-16-1EP_W4.40mm
- moved U7 47.9 mm to (27.9, -35.6), turned to 270 degrees
Connections:
- R3 pad 2: PWM1-D -> Net-(R3-Pad2)
- R34 pad 2: PWM2-D -> Net-(R34-Pad2)
- R4 pad 2: PWM2-D -> Net-(R4-Pad2)
- R41 pad 2: PWM1-D -> Net-(R41-Pad2)
- R5 pad 2: PWM1-D -> Net-(R5-Pad2)
- R6 pad 2: PWM2-D -> Net-(R6-Pad2)
- RS1 pad 1: PWM1-S -> Net-(RS1-Pad1)
- RS2 pad 1: PWM1-S -> Net-(RS2-Pad1)
- RS3 pad 1: PWM1-S -> Net-(RS3-Pad1)
- U7 pad 10: (no net) -> Net-(R5-Pad2)
- U7 pad 11: (no net) -> Net-(RS1-Pad1)
- U7 pad 13: VCC -> (no net)
- U7 pad 14: (no net) -> Net-(RS3-Pad1)
- U7 pad 15: (no net) -> Net-(R4-Pad2)
- U7 pad 16: (no net) -> PWM2
- U7 pad 2: PWM1-D -> Net-(R3-Pad2)
- U7 pad 3: PWM1-S -> Net-(RS3-Pad1)
- U7 pad 6: PWM1-S -> Net-(RS1-Pad1)
- U7 pad 7: PWM2-D -> Net-(R34-Pad2)
- U7 pad 9: (no net) -> PWM1
Routing:
- net VCC: track 232.9 -> 210.9 mm
