File: v_0.8/four_probe.sch (KiCad schematic (older format))
At the start: 75 parts, among them J1 Conn_01x13_Male, J2 RG, J3 Conn_01x13_Male, U1 LMC6482, U10 ADG704, U11 tmux1511, U2 AD623, U3 LMC6482, U4 AD623, U5 LMC6484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

Commit message: update
Parts:
- removed J1, J3: Conn_01x13_Male, Connector_PinHeader_2.54mm:PinHeader_1x13_P2.54mm_Vertical, symbol Connector:Conn_01x13_Male
- added J1: Conn_01x26_Male, Connector_PinHeader_2.54mm:PinHeader_1x26_P2.54mm_Vertical, symbol Connector:Conn_01x26_Male
- added J4: CONSMA001-SMD-G, digikey-footprints:RF_SMA_Receptical_Vertical_CONSMA001-SMD-G, symbol dk_Coaxial-Connectors-RF:CONSMA001-SMD-G
Connections:
- net GND: now also J1.25 (Pin_25)
- net GNDREF: now also J1.24 (Pin_24)
- net MUXGA: now also J1.8 (Pin_8)
- net MUXGB: now also J1.9 (Pin_9)
- net MUXRA: now also J1.6 (Pin_6)
- net MUXRB: now also J1.7 (Pin_7)
- net MUXVA: now also J1.4 (Pin_4)
- net MUXVB: now also J1.5 (Pin_5)
- net PWM1: now also J1.19 (Pin_19)
- net PWM2: now also J1.18 (Pin_18)
- net RGA: now also J1.14 (Pin_14)
- net RGB: now also J1.13 (Pin_13)
- net TIA: now also J1.1 (Pin_1)
- net TIB: now also J1.2 (Pin_2)
- net TIC: now also J1.3 (Pin_3)
- net V12A: now also J1.17 (Pin_17)
- net V12B: now also J1.16 (Pin_16)
- net V12C: now also J1.15 (Pin_15)
- net V23B: now also J1.10 (Pin_10), J1.11 (Pin_11)
- net V23C: now also J1.12 (Pin_12)
- net VCC: now also J1.26 (Pin_26)
- net VIN1: now also J1.23 (Pin_23)
- net VIN2: now also J1.22 (Pin_22)
- net VIN3: now also J1.21 (Pin_21)
- net VIN4: now also J1.20 (Pin_20)
Other:
- moved on the sheet: RF7, RF8, U6D

Commit message: update
Parts:
- added CU11: 0.1uF, Capacitor_SMD:C_0603_1608Metric, symbol four_probe-rescue:C
- added J3, J5, J6: CONSMA001-SMD-G, digikey-footprints:RF_SMA_Receptical_Vertical_CONSMA001-SMD-G, symbol dk_Coaxial-Connectors-RF:CONSMA001-SMD-G
- renumbered RL4A1 to RL4
Connections:
- net GND: now also J4.1, CU11.2, J3.1, J5.1, J6.1
- net P1: now also J4.2
- net P3: now also J5.2; no longer JP1.2 (Pin_2), U2.3 (+), U4.2 (-)
- net P4: now also J6.2
- net VCC: now also CU11.1
- new net P2: J3.2, JP1.2 (Pin_2), U2.3 (+), U4.2 (-)
Other:
- moved on the sheet: CU1, CU10, CU2, CU3, CU4, CU5, CU6, CU7, CU8, CU9, J4
