File: v_0.8/four_probe.kicad_pcb (KiCad board)
At the start: 2 copper layers, 74 parts, among them J1 Conn_02x13_Counter_Clockwise, J2 RG, U1 LMC6482, U10 ADG704, U11 adg1211, U2 AD623, U3 LMC6482, U4 AD623, U5 LMC6484, U6 LMC6484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

Commit message: update
Parts:
- added J4: CONSMA001-SMD-G, digikey-footprints:RF_SMA_Receptical_Vertical_CONSMA001-SMD-G, F.Cu at (8.89, 41.9)
- J1: value Conn_02x13_Counter_Clockwise -> Conn_01x26_Male; footprint Connector_PinSocket_2.54mm:PinSocket_1x26_P2.54mm_Vertical -> Connector_PinHeader_2.54mm:PinHeader_1x26_P2.54mm_Vertical
- U11, U7: value adg1211 -> tmux1511; footprint digikey-footprints:TSSOP-16-1EP_W4.40mm -> digikey-footprints:TSSOP-14_W4.4mm
- moved U6 172.5 mm to (-40.3, 84.8), turned to 270 degrees
- moved U8 166.6 mm to (-24.5, 82.7), turned to 270 degrees
- moved U5 140.7 mm to (-32.5, 63.4), turned to 270 degrees
- moved U3 114.3 mm to (-29.2, 45.0), turned to 270 degrees
- moved U4 101.7 mm to (-43.1, 32.1), turned to 270 degrees
- moved U2 91.9 mm to (-29.1, 29.0), turned to 270 degrees
- moved J1 83.2 mm to (0.00, 30.5), turned to 180 degrees
- moved U10 83.2 mm to (-40.8, 18.9), turned to 270 degrees
- moved U11 75.8 mm to (-24.2, 18.2), turned to 270 degrees
- moved U1 69.7 mm to (-30.4, 12.6), turned to 270 degrees
- moved JP1 67.4 mm to (82.5, 52.0)
- moved U7 63.8 mm to (-16.5, 10.2), turned to 180 degrees
- moved U9 48.7 mm to (-30.2, -3.05), turned to 270 degrees
- moved J2 27.6 mm to (74.9, 43.2), turned to 90 degrees
Connections:
- J1 pad 1: VCC -> TIA
- J1 pad 10: V12B -> V23B
- J1 pad 11: V12C -> V23B
- J1 pad 12: RGA -> V23C
- J1 pad 14: GNDREF -> RGA
- J1 pad 15: V23C -> V12C
- J1 pad 16: V23B -> V12B
- J1 pad 17: V23B -> V12A
- J1 pad 18: MUXGB -> PWM2
- J1 pad 19: MUXGA -> PWM1
- J1 pad 2: GND -> TIB
- J1 pad 20: MUXRB -> VIN4
- J1 pad 21: MUXRA -> VIN3
- J1 pad 22: MUXVB -> VIN2
- J1 pad 23: MUXVA -> VIN1
- J1 pad 24: TIC -> GNDREF
- J1 pad 25: TIB -> GND
- J1 pad 26: TIA -> VCC
- J1 pad 3: VIN1 -> TIC
- J1 pad 4: VIN2 -> MUXVA
- J1 pad 5: VIN3 -> MUXVB
- J1 pad 6: VIN4 -> MUXRA
- J1 pad 7: PWM1 -> MUXRB
- J1 pad 8: PWM2 -> MUXGA
- J1 pad 9: V12A -> MUXGB
- U11 pad 14: Net-(RS2-Pad1) -> VCC
- U11 pad 2: Net-(R41-Pad2) -> Net-(RS2-Pad1)
- U11 pad 3: Net-(RS2-Pad1) -> Net-(R41-Pad2)
- U11 pad 4: GND -> PWM2
- U11 pad 5: GND -> Net-(RS2-Pad1)
- U11 pad 6: (no net) -> Net-(R6-Pad2)
- U11 pad 7: (no net) -> GND
- U7 pad 10: Net-(R5-Pad2) -> PWM1
- U7 pad 11: Net-(RS1-Pad1) -> Net-(R34-Pad2)
- U7 pad 12: (no net) -> Net-(RS1-Pad1)
- U7 pad 13: (no net) -> PWM2
- U7 pad 14: Net-(RS3-Pad1) -> VCC
- U7 pad 2: Net-(R3-Pad2) -> Net-(RS3-Pad1)
- U7 pad 3: Net-(RS3-Pad1) -> Net-(R3-Pad2)
- U7 pad 4: GND -> PWM2
- U7 pad 5: GND -> Net-(RS3-Pad1)
- U7 pad 6: Net-(RS1-Pad1) -> Net-(R4-Pad2)
- U7 pad 7: Net-(R34-Pad2) -> GND
- U7 pad 8: PWM2 -> Net-(R5-Pad2)
- U7 pad 9: PWM1 -> Net-(RS1-Pad1)
Routing:
- net VIN3: track 1.20 -> 0.00 mm

Commit message: update
Parts:
- removed RL4A1: R, Resistor_SMD:R_0603_1608Metric
- added CU11: 0.1uF, Capacitor_SMD:C_0603_1608Metric, F.Cu at (177.4, 122.5)
- added J3: CONSMA001-SMD-G, digikey-footprints:RF_SMA_Receptical_Vertical_CONSMA001-SMD-G, F.Cu at (64.8, 125.1)
- added J5: CONSMA001-SMD-G, digikey-footprints:RF_SMA_Receptical_Vertical_CONSMA001-SMD-G, F.Cu at (64.8, 134.6)
- added J6: CONSMA001-SMD-G, digikey-footprints:RF_SMA_Receptical_Vertical_CONSMA001-SMD-G, F.Cu at (64.8, 144.1)
- added RL4: R, Resistor_SMD:R_0603_1608Metric, F.Cu at (73.7, 123.6)
- moved U11 230.9 mm to (177.4, 130.8), turned to 0 degrees
- moved U6 211.1 mm to (163.4, 140.3), turned to 0 degrees
- moved U7 193.7 mm to (118.5, 149.1)
- moved U8 188.4 mm to (158.9, 125.7), turned to 0 degrees
- moved CU6 186.4 mm to (163.2, 150.7)
- moved U5 180.6 mm to (133.7, 134.1), turned to 0 degrees
- moved U3 167.0 mm to (115.4, 128.5), turned to 0 degrees
- moved U10 163.8 mm to (80.8, 128.8), turned to 0 degrees
- moved U2 162.7 mm to (100.0, 128.0), turned to 0 degrees
- moved U4 162.5 mm to (78.2, 140.2), turned to 180 degrees
- moved CF2 161.7 mm to (177.1, 148.4)
- moved U9 161.3 mm to (80.6, 114.0), turned to 0 degrees
- moved C5 159.5 mm to (188.5, 148.7)
- moved C84 158.2 mm to (183.8, 142.4), turned to 0 degrees
- moved JRG4 156.5 mm to (155.6, 150.4)
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Connections:
- J4 pad 1: Net-(J4-Pad1) -> GND
- J4 pad 2: (no net) -> P1
- JP1 pad 2: P3 -> P2
- U2 pad 3: P3 -> P2
- U4 pad 2: P3 -> P2
Routing:
- net VCC: track 210.9 -> 46.8 mm
- net P1: track 0.00 -> 53.0 mm, vias 0 -> 3
- net P2: track 0.00 -> 41.9 mm, vias 0 -> 2
- net P4: track 0.00 -> 38.2 mm
- net P3: track 0.00 -> 33.0 mm, vias 0 -> 2
- net Net-(JRL4-Pad2): track 0.00 -> 30.6 mm, vias 0 -> 2
- net RL4: track 0.00 -> 22.5 mm
- net MUXRA: track 0.00 -> 19.2 mm, vias 0 -> 2
- net RGB: track 0.00 -> 17.3 mm
- net GND: track 181.1 -> 165.3 mm, vias 4 -> 13
- net RL2: track 0.00 -> 15.1 mm, vias 0 -> 2
- net VIND: track 0.00 -> 12.9 mm
- net RGA: track 0.00 -> 12.9 mm
- net GNDREF: track 0.00 -> 10.2 mm, vias 0 -> 2
- net RL3: track 0.00 -> 9.96 mm
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
Commit message: update
Parts:
- moved C5 67.9 mm to (122.9, 131.1)
- moved C84 63.3 mm to (120.9, 135.1), turned to 90 degrees
- moved J1 60.8 mm to (136.7, 106.7), turned to 270 degrees
- moved CF2 56.8 mm to (120.9, 140.2), turned to 90 degrees
- moved R41 54.8 mm to (122.9, 135.1), turned to 90 degrees
- moved RF6 53.1 mm to (119.9, 144.8), turned to 90 degrees
- moved JRG4 52.8 mm to (103.1, 145.3), turned to 270 degrees
- moved R6 51.6 mm to (134.6, 131.6), turned to 90 degrees
- moved CF6 50.3 mm to (127.5, 144.8), turned to 270 degrees
- moved RF2 49.7 mm to (122.9, 140.2), turned to 270 degrees
- moved U11 45.2 mm to (132.6, 124.5)
- moved CT4 41.9 mm to (108.7, 145.8), turned to 0 degrees
- moved RG4 41.8 mm to (108.7, 142.7)
- moved CT3 41.7 mm to (108.7, 139.2)
- moved CF5 41.7 mm to (116.3, 121.4), turned to 270 degrees
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Routing:
- net VCC: track 46.8 -> 245.1 mm, vias 2 -> 17
- net PWM1: track 0.00 -> 133.9 mm, vias 0 -> 4
- net GND: track 165.3 -> 292.6 mm, vias 13 -> 19
- net PWM2: track 0.00 -> 93.4 mm, vias 0 -> 2
- net GNDREF: track 10.2 -> 99.1 mm, vias 2 -> 9
- net TIB: track 0.00 -> 72.4 mm
- net Net-(U3-Pad6): track 0.00 -> 70.0 mm, vias 0 -> 2
- net P4: track 38.2 -> 103.4 mm
- net TIC: track 0.00 -> 60.7 mm, vias 0 -> 2
- net TIA: track 0.00 -> 58.3 mm, vias 0 -> 3
- net TG4: track 0.00 -> 39.9 mm
- net TG2: track 0.00 -> 36.5 mm, vias 0 -> 2
- net TG3: track 0.00 -> 35.3 mm, vias 0 -> 2
- net Net-(RS1-Pad1): track 0.00 -> 29.1 mm, vias 0 -> 4
- net Net-(R5-Pad2): track 0.00 -> 28.7 mm, vias 0 -> 2
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