File: v_0.9/four_probe.sch (KiCad schematic (older format))
At the start: 79 parts, among them J1 Conn_01x26_Male, J2 RG, J3 CONSMA001-SMD-G, J4 CONSMA001-SMD-G, J5 CONSMA001-SMD-G, J6 CONSMA001-SMD-G, U1 LMC6482, U10 ADG704, U11 tmux1511, U2 AD623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

Commit message: update
Parts:
- removed J1: Conn_01x26_Male, Connector_PinHeader_2.54mm:PinHeader_1x26_P2.54mm_Vertical, symbol Connector:Conn_01x26_Male
- added J1: Conn_01x30_Male, Connector_PinHeader_2.54mm:PinHeader_1x30_P2.54mm_Vertical, symbol Connector:Conn_01x30_Male
Connections:
- net GND: now also J1.25 (Pin_25)
- net GNDREF: now also J1.24 (Pin_24)
- net MUXGA: now also J1.8 (Pin_8)
- net MUXGB: now also J1.9 (Pin_9)
- net MUXRA: now also J1.6 (Pin_6)
- net MUXRB: now also J1.7 (Pin_7)
- net MUXVA: now also J1.4 (Pin_4)
- net MUXVB: now also J1.5 (Pin_5)
- net P1: now also J1.30 (Pin_30)
- net P2: now also J1.29 (Pin_29)
- net P3: now also J1.28 (Pin_28)
- net P4: now also J1.27 (Pin_27)
- net PWM1: now also J1.19 (Pin_19)
- net PWM2: now also J1.18 (Pin_18)
- net RGA: now also J1.14 (Pin_14)
- net RGB: now also J1.13 (Pin_13)
- net TIA: now also J1.1 (Pin_1)
- net TIB: now also J1.2 (Pin_2)
- net TIC: now also J1.3 (Pin_3)
- net V12A: now also J1.17 (Pin_17)
- net V12B: now also J1.16 (Pin_16)
- net V12C: now also J1.15 (Pin_15)
- net V23A: now also J1.12 (Pin_12)
- net V23B: now also J1.11 (Pin_11)
- net V23C: now also J1.10 (Pin_10)
- net VCC: now also J1.26 (Pin_26)
- net VIN1: now also J1.23 (Pin_23)
- net VIN2: now also J1.22 (Pin_22)
- net VIN3: now also J1.21 (Pin_21)
- net VIN4: now also J1.20 (Pin_20)
Other:
- moved on the sheet: JP1
Changed lines of the file:
@@
 L four_probe-rescue:Conn_01x04_Female JP1
 U 1 1 5AF5542B
-P 2400 6450
-F 0 "JP1" H 2400 6650 50  0000 C CNN
-F 1 "Conn_01x04_Female" H 2400 6150 50  0000 C CNN
-F 2 "Connector_PinSocket_2.54mm:PinSocket_1x04_P2.54mm_Vertical" H 2400 6450 50  0001 C CNN
-F 3 "" H 2400 6450 50  0001 C CNN
-	1    2400 6450
+P 2450 6450
+F 0 "JP1" H 2450 6650 50  0000 C CNN
+F 1 "Conn_01x04_Female" H 2450 6150 50  0000 C CNN
+F 2 "Connector_PinSocket_2.54mm:PinSocket_1x04_P2.54mm_Vertical" H 2450 6450 50  0001 C CNN
+F 3 "" H 2450 6450 50  0001 C CNN
+	1    2450 6450
 	1    0    0    -1
 $EndComp
@@
 Text GLabel 4400 5600 0    60   Input ~ 0
 P2
-Text GLabel 2200 6650 0    60   Input ~ 0
+Text GLabel 2250 6650 0    60   Input ~ 0
 PT4
-Text GLabel 2200 6550 0    60   Input ~ 0
+Text GLabel 2250 6550 0    60   Input ~ 0
 PT3
-Text GLabel 2200 6450 0    60   Input ~ 0
+Text GLabel 2250 6450 0    60   Input ~ 0
 PT2
-Text GLabel 2200 6350 0    60   Input ~ 0
+Text GLabel 2250 6350 0    60   Input ~ 0
 PT1
 Text GLabel 6200 5350 2    60   Input ~ 0
@@
 Connection ~ 11500 2400
 Connection ~ 11500 3150
-Wire Wire Line
-	15750 2400 15300 2400
-Wire Wire Line
-	15750 2300 15300 2300
 $Comp
 L four_probe-rescue:GND-power #PWR02
@@
 Text GLabel 15750 3600 0    60   Input ~ 0
 RGB
-$Comp
-L Connector:Conn_01x26_Male J1
-U 1 1 5D07D0A5
-P 15950 3600
-F 0 "J1" H 15922 3482 50  0000 R CNN
-F 1 "Conn_01x26_Male" H 15922 3573 50  0000 R CNN
-F 2 "Connector_PinHeader_2.54mm:PinHeader_1x26_P2.54mm_Vertical" H 15950 3600 50  0001 C CNN
-F 3 "~" H 15950 3600 50  0001 C CNN
-	1    15950 3600
-	-1   0    0    1
-$EndComp
 $Comp
 L four_probe-rescue:GNDREF-power #PWR0103
@@
 Text GLabel 15750 4600 0    60   Input ~ 0
 TIC
-Wire Wire Line
-	15750 2500 15050 2500
 $Comp
 L dk_Coaxial-Connectors-RF:CONSMA001-SMD-G J3
@@
 	1    0    0    -1
 $EndComp
+$Comp
+L Connector:Conn_01x30_Male J1
+U 1 1 5D1BAB9F
+P 15950 3400
+F 0 "J1" H 15922 3282 50  0000 R CNN
+F 1 "Conn_01x30_Male" H 15922 3373 50  0000 R CNN
+F 2 "Connector_PinHeader_2.54mm:PinHeader_1x30_P2.54mm_Vertical" H 15950 3400 50  0001 C CNN
+F 3 "~" H 15950 3400 50  0001 C CNN
+	1    15950 3400
+	-1   0    0    1
+$EndComp
+Text GLabel 15750 1900 0    60   Input ~ 0
+PT1
+Text GLabel 15750 2000 0    60   Input ~ 0
+PT2
+Text GLabel 15750 2100 0    60   Input ~ 0
+PT3
+Text GLabel 15750 2200 0    60   Input ~ 0
+PT4
+Wire Wire Line
+	15300 2300 15750 2300
+Wire Wire Line
+	15300 2400 15750 2400
+Wire Wire Line
+	15050 2500 15750 2500
 $EndSCHEMATC
