File: v_0.9/four_probe.sch (KiCad schematic (older format))
At the start: 79 parts, among them J1 Conn_01x30_Male, J2 RG, J3 CONSMA001-SMD-G, J4 CONSMA001-SMD-G, J5 CONSMA001-SMD-G, J6 CONSMA001-SMD-G, U1 LMC6482, U10 ADG704, U11 tmux1511, U2 AD623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

Commit message: update
Other:
- note added: "Four Probe v_0.9"
- note removed: "Four Probe v_0.8"
Changed lines of the file:
@@
 PROBES
 Text Notes 13050 9650 0    200  ~ 0
-Four Probe v_0.8
+Four Probe v_0.9
 Text Notes 13200 7850 0    60   ~ 0
 Switch for -VEXC

Commit message: update
Other:
- note added: "Probe Connectors"
- note removed: "Probes"
- moved on the sheet: J3, J4, J5, J6, JP1

Commit message: update
Connections:
- net GNDREF: now also J1.13 (Pin_13); no longer J1.24 (Pin_24)
- net MUXGA: now also J1.3 (Pin_3); no longer J1.8 (Pin_8)
- net MUXGB: now also J1.5 (Pin_5); no longer J1.9 (Pin_9)
- net MUXRA: now also J1.15 (Pin_15); no longer J1.6 (Pin_6)
- net MUXRB: now also J1.14 (Pin_14); no longer J1.7 (Pin_7)
- net MUXVA: now also J1.23 (Pin_23); no longer J1.4 (Pin_4)
- net MUXVB: now also J1.21 (Pin_21); no longer J1.5 (Pin_5)
- net P1: now also J1.27 (Pin_27); no longer J1.30 (Pin_30)
- net P2: now also J1.28 (Pin_28); no longer J1.29 (Pin_29)
- net P3: now also J1.29 (Pin_29); no longer J1.28 (Pin_28)
- net P4: now also J1.30 (Pin_30); no longer J1.27 (Pin_27)
- net PWM1: now also J1.10 (Pin_10); no longer J1.19 (Pin_19)
- net PWM2: now also J1.11 (Pin_11); no longer J1.18 (Pin_18)
- net RGA: now also J1.16 (Pin_16); no longer J1.14 (Pin_14)
- net RGB: now also J1.18 (Pin_18); no longer J1.13 (Pin_13)
- net TIA: now also J1.4 (Pin_4); no longer J1.1 (Pin_1)
- net TIB: now also J1.9 (Pin_9); no longer J1.2 (Pin_2)
- net TIC: now also J1.8 (Pin_8); no longer J1.3 (Pin_3)
- net V12A: now also J1.12 (Pin_12); no longer J1.17 (Pin_17)
- net V12B: now also J1.6 (Pin_6); no longer J1.16 (Pin_16)
- net V12C: now also J1.2 (Pin_2); no longer J1.15 (Pin_15)
- net V23A: now also J1.17 (Pin_17); no longer J1.12 (Pin_12)
- net V23B: now also J1.1 (Pin_1); no longer J1.11 (Pin_11)
- net V23C: now also J1.7 (Pin_7); no longer J1.10 (Pin_10)
- net VIN1: now also J1.22 (Pin_22); no longer J1.23 (Pin_23)
- net VIN2: now also J1.20 (Pin_20); no longer J1.22 (Pin_22)
- net VIN3: now also J1.24 (Pin_24); no longer J1.21 (Pin_21)
- net VIN4: now also J1.19 (Pin_19); no longer J1.20 (Pin_20)
Changed lines of the file:
@@
 	1    0    0    -1
 $EndComp
-Text GLabel 15500 3800 0    60   Input ~ 0
-V12C
 Text GLabel 15500 3600 0    60   Input ~ 0
-V12A
-Text GLabel 15500 3700 0    60   Input ~ 0
-V12B
+V23A
+Text GLabel 15500 5200 0    60   Input ~ 0
+V23B
+Text GLabel 15500 4600 0    60   Input ~ 0
+V23C
+Text GLabel 15500 4800 0    60   Input ~ 0
+MUXGB
+Text GLabel 15500 5000 0    60   Input ~ 0
+MUXGA
+Text GLabel 15500 3200 0    60   Input ~ 0
+MUXVB
 Text GLabel 15500 3000 0    60   Input ~ 0
-VIN1
-Text GLabel 15500 3100 0    60   Input ~ 0
-VIN2
-Text GLabel 15500 3200 0    60   Input ~ 0
-VIN3
-Text GLabel 15500 3300 0    60   Input ~ 0
-VIN4
-Text GLabel 15500 3400 0    60   Input ~ 0
-PWM1
-Text GLabel 15500 3500 0    60   Input ~ 0
-PWM2
-Text GLabel 15500 3900 0    60   Input ~ 0
-RGA
-Text GLabel 15500 4000 0    60   Input ~ 0
-RGB
-$Comp
-L four_probe-rescue:GNDREF-power #PWR0103
-U 1 1 5BD6F7F4
-P 14800 2900
-F 0 "#PWR0103" H 14800 2650 50  0001 C CNN
-F 1 "GNDREF" H 14800 2750 50  0000 C CNN
-F 2 "" H 14800 2900 50  0001 C CNN
-F 3 "" H 14800 2900 50  0001 C CNN
-	1    14800 2900
-	-1   0    0    1
-$EndComp
-Text GLabel 15500 4100 0    60   Input ~ 0
-V23A
-Text GLabel 15500 4200 0    60   Input ~ 0
-V23B
-Text GLabel 15500 4300 0    60   Input ~ 0
-V23C
-Text GLabel 15500 4400 0    60   Input ~ 0
-MUXGB
+MUXVA
+Text GLabel 15500 4900 0    60   Input ~ 0
+TIA
 Text GLabel 15500 4500 0    60   Input ~ 0
-MUXGA
-Text GLabel 15500 4600 0    60   Input ~ 0
-MUXRB
-Text GLabel 15500 4700 0    60   Input ~ 0
-MUXRA
-Text GLabel 15500 4800 0    60   Input ~ 0
-MUXVB
-Text GLabel 15500 4900 0    60   Input ~ 0
-MUXVA
-Text GLabel 15500 5100 0    60   Input ~ 0
-TIB
-Text GLabel 15500 5200 0    60   Input ~ 0
-TIA
-Text GLabel 15500 5000 0    60   Input ~ 0
 TIC
 $Comp
@@
 	-1   0    0    1
 $EndComp
+Text GLabel 15500 2600 0    60   Input ~ 0
+PT1
+Text GLabel 15500 2500 0    60   Input ~ 0
+PT2
+Text GLabel 15500 2400 0    60   Input ~ 0
+PT3
 Text GLabel 15500 2300 0    60   Input ~ 0
-PT1
-Text GLabel 15500 2400 0    60   Input ~ 0
-PT2
-Text GLabel 15500 2500 0    60   Input ~ 0
-PT3
-Text GLabel 15500 2600 0    60   Input ~ 0
 PT4
 Wire Wire Line
@@
 	15050 2800 15500 2800
 Wire Wire Line
-	14800 2900 15500 2900
+	15500 4000 14950 4000
+Text GLabel 15500 3400 0    60   Input ~ 0
+VIN4
+Text GLabel 15500 2900 0    60   Input ~ 0
+VIN3
+Text GLabel 15500 3300 0    60   Input ~ 0
+VIN2
+Text GLabel 15500 3100 0    60   Input ~ 0
+VIN1
+Text GLabel 15500 3800 0    60   Input ~ 0
+MUXRA
+Text GLabel 15500 3900 0    60   Input ~ 0
+MUXRB
+$Comp
+L four_probe-rescue:GNDREF-power #PWR0103
+U 1 1 5BD6F7F4
+P 14950 4000
+F 0 "#PWR0103" H 14950 3750 50  0001 C CNN
+F 1 "GNDREF" H 14950 3850 50  0000 C CNN
+F 2 "" H 14950 4000 50  0001 C CNN
+F 3 "" H 14950 4000 50  0001 C CNN
+	1    14950 4000
+	1    0    0    -1
+$EndComp
+Text GLabel 15500 3500 0    60   Input ~ 0
+RGB
+Text GLabel 15500 3700 0    60   Input ~ 0
+RGA
+Text GLabel 15500 4200 0    60   Input ~ 0
+PWM2
+Text GLabel 15500 4300 0    60   Input ~ 0
+PWM1
+Text GLabel 15500 4700 0    60   Input ~ 0
+V12B
+Text GLabel 15500 4100 0    60   Input ~ 0
+V12A
+Text GLabel 15500 5100 0    60   Input ~ 0
+V12C
+Text GLabel 15500 4400 0    60   Input ~ 0
+TIB
 $EndSCHEMATC

Commit message: update
Connections:
- net GNDREF: now also J1.14 (Pin_14); no longer J1.13 (Pin_13)
- net MUXGB: now also J1.4 (Pin_4); no longer J1.5 (Pin_5)
- net MUXRB: now also J1.13 (Pin_13); no longer J1.14 (Pin_14)
- net MUXVA: now also J1.24 (Pin_24); no longer J1.23 (Pin_23)
- net TIA: now also J1.5 (Pin_5); no longer J1.4 (Pin_4)
- net VIN1: now also J1.23 (Pin_23); no longer J1.22 (Pin_22)
- net VIN3: now also J1.22 (Pin_22); no longer J1.24 (Pin_24)
Changed lines of the file:
@@
 Text GLabel 15500 4600 0    60   Input ~ 0
 V23C
-Text GLabel 15500 4800 0    60   Input ~ 0
+Text GLabel 15500 4900 0    60   Input ~ 0
 MUXGB
 Text GLabel 15500 5000 0    60   Input ~ 0
@@
 Text GLabel 15500 3200 0    60   Input ~ 0
 MUXVB
-Text GLabel 15500 3000 0    60   Input ~ 0
+Text GLabel 15500 2900 0    60   Input ~ 0
 MUXVA
-Text GLabel 15500 4900 0    60   Input ~ 0
+Text GLabel 15500 4800 0    60   Input ~ 0
 TIA
 Text GLabel 15500 4500 0    60   Input ~ 0
@@
 Wire Wire Line
 	15050 2800 15500 2800
-Wire Wire Line
-	15500 4000 14950 4000
 Text GLabel 15500 3400 0    60   Input ~ 0
 VIN4
-Text GLabel 15500 2900 0    60   Input ~ 0
+Text GLabel 15500 3100 0    60   Input ~ 0
 VIN3
 Text GLabel 15500 3300 0    60   Input ~ 0
 VIN2
-Text GLabel 15500 3100 0    60   Input ~ 0
+Text GLabel 15500 3000 0    60   Input ~ 0
 VIN1
 Text GLabel 15500 3800 0    60   Input ~ 0
 MUXRA
-Text GLabel 15500 3900 0    60   Input ~ 0
+Text GLabel 15500 4000 0    60   Input ~ 0
 MUXRB
 $Comp
 L four_probe-rescue:GNDREF-power #PWR0103
 U 1 1 5BD6F7F4
-P 14950 4000
-F 0 "#PWR0103" H 14950 3750 50  0001 C CNN
-F 1 "GNDREF" H 14950 3850 50  0000 C CNN
-F 2 "" H 14950 4000 50  0001 C CNN
-F 3 "" H 14950 4000 50  0001 C CNN
-	1    14950 4000
+P 14950 3900
+F 0 "#PWR0103" H 14950 3650 50  0001 C CNN
+F 1 "GNDREF" H 14950 3750 50  0000 C CNN
+F 2 "" H 14950 3900 50  0001 C CNN
+F 3 "" H 14950 3900 50  0001 C CNN
+	1    14950 3900
 	1    0    0    -1
 $EndComp
@@
 Text GLabel 15500 4400 0    60   Input ~ 0
 TIB
+Wire Wire Line
+	15500 3900 14950 3900
 $EndSCHEMATC

Commit message: update
Parts:
- removed J1: Conn_01x30_Male, Connector_PinHeader_2.54mm:PinHeader_1x30_P2.54mm_Vertical, symbol Connector:Conn_01x30_Male
- added J1: Conn_01x32_Male, Connector_PinHeader_2.54mm:PinHeader_1x32_P2.54mm_Vertical, symbol Connector:Conn_01x32_Male
- renumbered JRV12G1 to JR1, JRG4 to JR4, RV12G1 to RG12
Connections:
- net GND: now also J1.27 (Pin_27)
- net GNDREF: now also J1.14 (Pin_14)
- net MUXGA: now also J1.3 (Pin_3)
- net MUXGB: now also J1.4 (Pin_4)
- net MUXRA: now also J1.15 (Pin_15)
- net MUXRB: now also J1.13 (Pin_13)
- net MUXVA: now also J1.26 (Pin_26)
- net MUXVB: now also J1.23 (Pin_23)
- net P1: now also J1.29 (Pin_29)
- net P2: now also J1.30 (Pin_30)
- net P3: now also J1.31 (Pin_31)
- net P4: now also J1.32 (Pin_32)
- net PWM1: now also J1.10 (Pin_10)
- net PWM2: now also J1.11 (Pin_11)
- net TIA: now also J1.5 (Pin_5)
- net TIB: now also J1.9 (Pin_9)
- net TIC: now also J1.8 (Pin_8)
- net V12A: now also J1.12 (Pin_12)
- net V12B: now also J1.6 (Pin_6)
- net V12C: now also J1.2 (Pin_2)
- net V23A: now also J1.16 (Pin_16)
- net V23B: now also J1.1 (Pin_1)
- net V23C: now also J1.7 (Pin_7)
- net VCC: now also J1.28 (Pin_28)
- net VIN1: now also J1.25 (Pin_25)
- net VIN2: now also J1.22 (Pin_22)
- net VIN3: now also J1.24 (Pin_24)
- net VIN4: now also J1.21 (Pin_21)
- net RG12B: now reaches JR1.1 (Pin_1), RG12.1, U2.8 (Rg)
- net RG12B: now also J1.17 (Pin_17)
- net RG12A: now reaches JR1.2 (Pin_2), RG12.2, U2.1 (Rg)
- net RG12A: now also J1.18 (Pin_18)
- net RGA renamed RG23A
- net RG23A: now also J1.20 (Pin_20)
- net RGB renamed RG23B
- net RG23B: now also J1.19 (Pin_19)
Changed lines of the file:
@@
 $EndComp
 $Comp
-L four_probe-rescue:R RV12G1
+L four_probe-rescue:R RG12
 U 1 1 5AE5B09A
 P 5000 2100
-F 0 "RV12G1" V 5100 2100 50  0000 C CNN
+F 0 "RG12" V 5100 2100 50  0000 C CNN
 F 1 "R" V 5000 2100 50  0000 C CNN
 F 2 "Resistor_SMD:R_0603_1608Metric" V 4930 2100 50  0001 C CNN
@@
 Should match capacitors to gain resistors
 $Comp
-L four_probe-rescue:Conn_01x02 JRG4
+L four_probe-rescue:Conn_01x02 JR4
 U 1 1 5AFF8263
 P 12750 6100
-F 0 "JRG4" H 12750 6200 50  0000 C CNN
+F 0 "JR4" H 12750 6200 50  0000 C CNN
 F 1 "Conn_01x02" H 12750 5900 50  0000 C CNN
 F 2 "Connector_PinSocket_2.54mm:PinSocket_1x02_P2.54mm_Vertical" H 12750 6100 50  0001 C CNN
@@
 $EndComp
 $Comp
-L four_probe-rescue:Conn_01x02 JRV12G1
+L four_probe-rescue:Conn_01x02 JR1
 U 1 1 5B0046BD
 P 4300 2250
-F 0 "JRV12G1" H 4250 2050 50  0000 C CNN
+F 0 "JR1" H 4250 2050 50  0000 C CNN
 F 1 "Conn_01x02" H 4150 2350 50  0000 C CNN
 F 2 "Connector_PinSocket_2.54mm:PinSocket_1x02_P2.54mm_Vertical" H 4300 2250 50  0001 C CNN
@@
 	5200 2250 5200 2200
 Wire Wire Line
-	4500 2250 5000 2250
-Wire Wire Line
-	4500 1950 5000 1950
+	4500 2250 4750 2250
+Wire Wire Line
+	4500 1950 4750 1950
 Wire Wire Line
 	5200 1950 5200 2000
@@
 Wire Wire Line
 	4900 5650 4950 5650
-Text GLabel 4900 5750 0    60   Input ~ 0
-RGA
-Text GLabel 4900 5950 0    60   Input ~ 0
-RGB
 Wire Wire Line
 	4900 5650 4900 5750
@@
 L four_probe-rescue:GND-power #PWR02
 U 1 1 5AC58D11
-P 15050 2800
-F 0 "#PWR02" H 15050 2550 50  0001 C CNN
-F 1 "GND" H 15050 2650 50  0000 C CNN
-F 2 "" H 15050 2800 50  0001 C CNN
-F 3 "" H 15050 2800 50  0001 C CNN
-	1    15050 2800
+P 15150 2800
+F 0 "#PWR02" H 15150 2550 50  0001 C CNN
+F 1 "GND" H 15150 2650 50  0000 C CNN
+F 2 "" H 15150 2800 50  0001 C CNN
+F 3 "" H 15150 2800 50  0001 C CNN
+	1    15150 2800
 	1    0    0    -1
 $EndComp
@@
 L four_probe-rescue:VCC-power #PWR01
 U 1 1 5AC58CD2
-P 15050 2700
-F 0 "#PWR01" H 15050 2550 50  0001 C CNN
-F 1 "VCC" H 15050 2850 50  0000 C CNN
-F 2 "" H 15050 2700 50  0001 C CNN
-F 3 "" H 15050 2700 50  0001 C CNN
-	1    15050 2700
-	1    0    0    -1
-$EndComp
-Text GLabel 15500 3600 0    60   Input ~ 0
+P 15150 2700
+F 0 "#PWR01" H 15150 2550 50  0001 C CNN
+F 1 "VCC" H 15150 2850 50  0000 C CNN
+F 2 "" H 15150 2700 50  0001 C CNN
+F 3 "" H 15150 2700 50  0001 C CNN
+	1    15150 2700
+	1    0    0    -1
+$EndComp
+Text GLabel 15600 3900 0    60   Input ~ 0
 V23A
-Text GLabel 15500 5200 0    60   Input ~ 0
+Text GLabel 15600 5400 0    60   Input ~ 0
 V23B
-Text GLabel 15500 4600 0    60   Input ~ 0
+Text GLabel 15600 4800 0    60   Input ~ 0
 V23C
-Text GLabel 15500 4900 0    60   Input ~ 0
+Text GLabel 15600 5100 0    60   Input ~ 0
 MUXGB
-Text GLabel 15500 5000 0    60   Input ~ 0
+Text GLabel 15600 5200 0    60   Input ~ 0
 MUXGA
-Text GLabel 15500 3200 0    60   Input ~ 0
+Text GLabel 15600 3200 0    60   Input ~ 0
 MUXVB
-Text GLabel 15500 2900 0    60   Input ~ 0
+Text GLabel 15600 2900 0    60   Input ~ 0
 MUXVA
-Text GLabel 15500 4800 0    60   Input ~ 0
+Text GLabel 15600 5000 0    60   Input ~ 0
 TIA
-Text GLabel 15500 4500 0    60   Input ~ 0
+Text GLabel 15600 4700 0    60   Input ~ 0
 TIC
 $Comp
@@
 	1    0    0    -1
 $EndComp
-$Comp
-L Connector:Conn_01x30_Male J1
-U 1 1 5D1BAB9F
-P 15700 3800
-F 0 "J1" H 15672 3682 50  0000 R CNN
-F 1 "Conn_01x30_Male" H 15672 3773 50  0000 R CNN
-F 2 "Connector_PinHeader_2.54mm:PinHeader_1x30_P2.54mm_Vertical" H 15700 3800 50  0001 C CNN
-F 3 "~" H 15700 3800 50  0001 C CNN
-	1    15700 3800
-	-1   0    0    1
-$EndComp
-Text GLabel 15500 2600 0    60   Input ~ 0
+Text GLabel 15600 2600 0    60   Input ~ 0
 PT1
-Text GLabel 15500 2500 0    60   Input ~ 0
+Text GLabel 15600 2500 0    60   Input ~ 0
 PT2
-Text GLabel 15500 2400 0    60   Input ~ 0
+Text GLabel 15600 2400 0    60   Input ~ 0
 PT3
-Text GLabel 15500 2300 0    60   Input ~ 0
+Text GLabel 15600 2300 0    60   Input ~ 0
 PT4
 Wire Wire Line
-	15050 2700 15500 2700
-Wire Wire Line
-	15050 2800 15500 2800
-Text GLabel 15500 3400 0    60   Input ~ 0
+	15150 2700 15600 2700
+Wire Wire Line
+	15150 2800 15600 2800
+Text GLabel 15600 3400 0    60   Input ~ 0
 VIN4
-Text GLabel 15500 3100 0    60   Input ~ 0
+Text GLabel 15600 3100 0    60   Input ~ 0
 VIN3
-Text GLabel 15500 3300 0    60   Input ~ 0
+Text GLabel 15600 3300 0    60   Input ~ 0
 VIN2
-Text GLabel 15500 3000 0    60   Input ~ 0
+Text GLabel 15600 3000 0    60   Input ~ 0
 VIN1
-Text GLabel 15500 3800 0    60   Input ~ 0
+Text GLabel 15600 4000 0    60   Input ~ 0
 MUXRA
-Text GLabel 15500 4000 0    60   Input ~ 0
+Text GLabel 15600 4200 0    60   Input ~ 0
 MUXRB
 $Comp
 L four_probe-rescue:GNDREF-power #PWR0103
 U 1 1 5BD6F7F4
-P 14950 3900
-F 0 "#PWR0103" H 14950 3650 50  0001 C CNN
-F 1 "GNDREF" H 14950 3750 50  0000 C CNN
-F 2 "" H 14950 3900 50  0001 C CNN
-F 3 "" H 14950 3900 50  0001 C CNN
-	1    14950 3900
-	1    0    0    -1
-$EndComp
-Text GLabel 15500 3500 0    60   Input ~ 0
-RGB
-Text GLabel 15500 3700 0    60   Input ~ 0
-RGA
-Text GLabel 15500 4200 0    60   Input ~ 0
+P 15050 4100
+F 0 "#PWR0103" H 15050 3850 50  0001 C CNN
+F 1 "GNDREF" H 15050 3950 50  0000 C CNN
+F 2 "" H 15050 4100 50  0001 C CNN
+F 3 "" H 15050 4100 50  0001 C CNN
+	1    15050 4100
+	1    0    0    -1
+$EndComp
+Text GLabel 15600 4400 0    60   Input ~ 0
 PWM2
-Text GLabel 15500 4300 0    60   Input ~ 0
+Text GLabel 15600 4500 0    60   Input ~ 0
 PWM1
-Text GLabel 15500 4700 0    60   Input ~ 0
+Text GLabel 15600 4900 0    60   Input ~ 0
 V12B
-Text GLabel 15500 4100 0    60   Input ~ 0
+Text GLabel 15600 4300 0    60   Input ~ 0
 V12A
-Text GLabel 15500 5100 0    60   Input ~ 0
+Text GLabel 15600 5300 0    60   Input ~ 0
 V12C
-Text GLabel 15500 4400 0    60   Input ~ 0
+Text GLabel 15600 4600 0    60   Input ~ 0
 TIB
 Wire Wire Line
-	15500 3900 14950 3900
+	15600 4100 15050 4100
+Text GLabel 15600 3600 0    60   Input ~ 0
+RG23B
+Text GLabel 15600 3500 0    60   Input ~ 0
+RG23A
+Text GLabel 4900 5950 0    60   Input ~ 0
+RG23B
+Text GLabel 4900 5750 0    60   Input ~ 0
+RG23A
+Text GLabel 4750 1750 0    60   Input ~ 0
+RG12A
+Wire Wire Line
+	4750 1750 4750 1950
+Connection ~ 4750 1950
+Wire Wire Line
+	4750 1950 5000 1950
+Text GLabel 4750 2550 0    60   Input ~ 0
+RG12B
+Wire Wire Line
+	4750 2550 4750 2250
+Connection ~ 4750 2250
+Wire Wire Line
+	4750 2250 5000 2250
+Text GLabel 15600 3700 0    60   Input ~ 0
+RG12A
+Text GLabel 15600 3800 0    60   Input ~ 0
+RG12B
+$Comp
+L Connector:Conn_01x32_Male J1
+U 1 1 5D4F7A91
+P 15800 3900
+F 0 "J1" H 15772 3782 50  0000 R CNN
+F 1 "Conn_01x32_Male" H 15772 3873 50  0000 R CNN
+F 2 "Connector_PinHeader_2.54mm:PinHeader_1x32_P2.54mm_Vertical" H 15800 3900 50  0001 C CNN
+F 3 "~" H 15800 3900 50  0001 C CNN
+	1    15800 3900
+	-1   0    0    1
+$EndComp
 $EndSCHEMATC

Commit message: update
Parts:
- renumbered RV23G1 to RG23
Changed lines of the file:
@@
 R_test
-$Comp
-L four_probe-rescue:R RV23G1
-U 1 1 5ACBDA2E
-P 5100 5800
-F 0 "RV23G1" V 5200 5800 50  0000 C CNN
-F 1 "R" V 5100 5800 50  0000 C CNN
-F 2 "Resistor_SMD:R_0603_1608Metric" V 5030 5800 50  0001 C CNN
-F 3 "" H 5100 5800 50  0001 C CNN
-	1    5100 5800
-	-1   0    0    1
-$EndComp
 $Comp
 L four_probe-rescue:VCC-power #PWR017
@@
 	-1   0    0    1
 $EndComp
+$Comp
+L four_probe-rescue:R RG23
+U 1 1 5ACBDA2E
+P 5100 5800
+F 0 "RG23" V 5200 5800 50  0000 C CNN
+F 1 "R" V 5100 5800 50  0000 C CNN
+F 2 "Resistor_SMD:R_0603_1608Metric" V 5030 5800 50  0001 C CNN
+F 3 "" H 5100 5800 50  0001 C CNN
+	1    5100 5800
+	-1   0    0    1
+$EndComp
