File: v_0.9/four_probe.kicad_pcb (KiCad board)
At the start: 2 copper layers, 79 parts, among them J1 Conn_01x26_Male, J2 RG, J3 CONSMA001-SMD-G, J4 CONSMA001-SMD-G, J5 CONSMA001-SMD-G, J6 CONSMA001-SMD-G, U1 LMC6482, U10 ADG704, U11 tmux1511, U2 AD623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

Commit message: update
Parts:
- J1: value Conn_01x26_Male -> Conn_01x30_Male; footprint Connector_PinHeader_2.54mm:PinHeader_1x26_P2.54mm_Vertical -> Connector_PinHeader_2.54mm:PinHeader_1x30_P2.54mm_Vertical; moved to B.Cu
- moved U11 35.4 mm to (103.6, 131.1)
- moved R6 29.9 mm to (108.2, 137.2)
- moved JP1 27.6 mm to (70.6, 144.3), turned to 180 degrees
- moved R5 25.7 mm to (121.4, 143.8), turned to 180 degrees
- moved CU11 25.6 mm to (111.8, 117.3)
- moved RF4 25.4 mm to (134.6, 119.9), turned to 90 degrees
- moved C1 23.4 mm to (125.5, 138.2)
- moved R4 22.9 mm to (128.0, 127.5), turned to 0 degrees
- moved C3 22.9 mm to (115.8, 114.3), turned to 90 degrees
- moved CT3 21.9 mm to (132.1, 128.0)
- moved RG4 21.9 mm to (132.1, 131.6)
- moved C50 21.9 mm to (127.5, 134.1)
- moved CF3 21.6 mm to (131.6, 119.9), turned to 270 degrees
- moved JRG4 21.3 mm to (128.5, 144.3)
- moved CT1 20.8 mm to (136.7, 131.1)
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Other:
- board outline added: 80.8 x 45.7 mm

Commit message: update
Parts:
- moved RS3 4.60 mm to (97.5, 130.0)
- moved CG1 3.59 mm to (97.5, 126.5)
- moved J2 3.05 mm to (84.8, 144.3), turned to 270 degrees
- moved CU9 2.27 mm to (72.6, 111.3), turned to 90 degrees
- moved CU4 2.03 mm to (76.0, 139.2)
- moved JRL4 1.14 mm to (91.4, 135.6)
- moved RS1 1.14 mm to (91.4, 141.7)
- moved CG2 1.02 mm to (91.4, 145.8), turned to 270 degrees
Changed lines of the file:
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@@
   )
   (module Connector_PinSocket_2.54mm:PinSocket_1x02_P2.54mm_Vertical (layer F.Cu)
-    (at 90.424 136.144)
+    (at 91.44 135.636)
     (descr "Through hole straight socket strip, 1x02, 2.54mm pitch, single row (from Kicad 4.0.7), script generated")
     (tags "Through hole socket strip THT 1x02 2.54mm single row")
@@
   )
   (module Capacitor_SMD:C_0603_1608Metric (layer F.Cu)
-    (at 98.044 130.048)
+    (at 97.536 126.492)
     (descr "Capacitor SMD 0603 (1608 Metric), square (rectangular) end terminal, IPC_7351 nominal, (Body size source: http://www.tortai-tech.com/upload/download/2011102023233369053.pdf), generated with kicad-footprint-generator")
     (tags capacitor)
@@
   )
   (module Capacitor_SMD:C_0603_1608Metric (layer F.Cu)
-    (at 90.424 145.796 90)
+    (at 91.44 145.796 270)
     (descr "Capacitor SMD 0603 (1608 Metric), square (rectangular) end terminal, IPC_7351 nominal, (Body size source: http://www.tortai-tech.com/upload/download/2011102023233369053.pdf), generated with kicad-footprint-generator")
     (tags capacitor)
@@
     (fp_line (start -0.8 -0.4) (end 0.8 -0.4) (layer F.Fab) (width 0.1))
     (fp_line (start -0.8 0.4) (end -0.8 -0.4) (layer F.Fab) (width 0.1))
-    (pad 2 smd roundrect (at 0.7875 0 90) (size 0.875 0.95) (layers F.Cu F.Paste F.Mask) (roundrect_rratio 0.25)
+    (pad 2 smd roundrect (at 0.7875 0 270) (size 0.875 0.95) (layers F.Cu F.Paste F.Mask) (roundrect_rratio 0.25)
       (net 20 GND))
-    (pad 1 smd roundrect (at -0.7875 0 90) (size 0.875 0.95) (layers F.Cu F.Paste F.Mask) (roundrect_rratio 0.25)
+    (pad 1 smd roundrect (at -0.7875 0 270) (size 0.875 0.95) (layers F.Cu F.Paste F.Mask) (roundrect_rratio 0.25)
       (net 21 VCC))
     (model ${KISYS3DMOD}/Capacitor_SMD.3dshapes/C_0603_1608Metric.wrl
@@
   )
   (module Capacitor_SMD:C_0603_1608Metric (layer F.Cu)
-    (at 75.9715 141.224 180)
+    (at 75.9715 139.192 180)
     (descr "Capacitor SMD 0603 (1608 Metric), square (rectangular) end terminal, IPC_7351 nominal, (Body size source: http://www.tortai-tech.com/upload/download/2011102023233369053.pdf), generated with kicad-footprint-generator")
     (tags capacitor)
@@
   )
   (module Capacitor_SMD:C_0603_1608Metric (layer F.Cu)
-    (at 70.612 112.268 180)
-    (descr "Capacitor SMD 0603 (1608 Metric), square (rectangular) end terminal, IPC_7351 nominal, (Body size source: http://www.tortai-tech.com/upload/download/2011102023233369053.pdf), generated with kicad-footprint-generator")
-    (tags capacitor)
-    (attr smd)
-    (fp_text reference CU9 (at 0 -1.43) (layer F.SilkS)
-      (effects (font (size 1 1) (thickness 0.15)))
-    )
-    (fp_text value 0.1uF (at 0 1.43) (layer F.Fab)
-      (effects (font (size 1 1) (thickness 0.15)))
-    )
-    (fp_line (start -0.8 0.4) (end -0.8 -0.4) (layer F.Fab) (width 0.1))
-    (fp_line (start -0.8 -0.4) (end 0.8 -0.4) (layer F.Fab) (width 0.1))
-    (fp_line (start 0.8 -0.4) (end 0.8 0.4) (layer F.Fab) (width 0.1))
-    (fp_line (start 0.8 0.4) (end -0.8 0.4) (layer F.Fab) (width 0.1))
-    (fp_line (start -0.162779 -0.51) (end 0.162779 -0.51) (layer F.SilkS) (width 0.12))
-    (fp_line (start -0.162779 0.51) (end 0.162779 0.51) (layer F.SilkS) (width 0.12))
-    (fp_line (start -1.48 0.73) (end -1.48 -0.73) (layer F.CrtYd) (width 0.05))
-    (fp_line (start -1.48 -0.73) (end 1.48 -0.73) (layer F.CrtYd) (width 0.05))
-    (fp_line (start 1.48 -0.73) (end 1.48 0.73) (layer F.CrtYd) (width 0.05))
-    (fp_line (start 1.48 0.73) (end -1.48 0.73) (layer F.CrtYd) (width 0.05))
-    (fp_text user %R (at 0 0) (layer F.Fab)
-      (effects (font (size 0.4 0.4) (thickness 0.06)))
-    )
-    (pad 1 smd roundrect (at -0.7875 0 180) (size 0.875 0.95) (layers F.Cu F.Paste F.Mask) (roundrect_rratio 0.25)
+    (at 72.644 111.252 90)
+    (descr "Capacitor SMD 0603 (1608 Metric), square (rectangular) end terminal, IPC_7351 nominal, (Body size source: http://www.tortai-tech.com/upload/download/2011102023233369053.pdf), generated with kicad-footprint-generator")
+    (tags capacitor)
+    (attr smd)
+    (fp_text reference CU9 (at 0 -1.43 90) (layer F.SilkS)
+      (effects (font (size 1 1) (thickness 0.15)))
+    )
+    (fp_text value 0.1uF (at 0 1.43 90) (layer F.Fab)
+      (effects (font (size 1 1) (thickness 0.15)))
+    )
+    (fp_line (start -0.8 0.4) (end -0.8 -0.4) (layer F.Fab) (width 0.1))
+    (fp_line (start -0.8 -0.4) (end 0.8 -0.4) (layer F.Fab) (width 0.1))
+    (fp_line (start 0.8 -0.4) (end 0.8 0.4) (layer F.Fab) (width 0.1))
+    (fp_line (start 0.8 0.4) (end -0.8 0.4) (layer F.Fab) (width 0.1))
+    (fp_line (start -0.162779 -0.51) (end 0.162779 -0.51) (layer F.SilkS) (width 0.12))
+    (fp_line (start -0.162779 0.51) (end 0.162779 0.51) (layer F.SilkS) (width 0.12))
+    (fp_line (start -1.48 0.73) (end -1.48 -0.73) (layer F.CrtYd) (width 0.05))
+    (fp_line (start -1.48 -0.73) (end 1.48 -0.73) (layer F.CrtYd) (width 0.05))
+    (fp_line (start 1.48 -0.73) (end 1.48 0.73) (layer F.CrtYd) (width 0.05))
+    (fp_line (start 1.48 0.73) (end -1.48 0.73) (layer F.CrtYd) (width 0.05))
+    (fp_text user %R (at 0 0 90) (layer F.Fab)
+      (effects (font (size 0.4 0.4) (thickness 0.06)))
+    )
+    (pad 1 smd roundrect (at -0.7875 0 90) (size 0.875 0.95) (layers F.Cu F.Paste F.Mask) (roundrect_rratio 0.25)
       (net 21 VCC))
-    (pad 2 smd roundrect (at 0.7875 0 180) (size 0.875 0.95) (layers F.Cu F.Paste F.Mask) (roundrect_rratio 0.25)
+    (pad 2 smd roundrect (at 0.7875 0 90) (size 0.875 0.95) (layers F.Cu F.Paste F.Mask) (roundrect_rratio 0.25)
       (net 20 GND))
     (model ${KISYS3DMOD}/Capacitor_SMD.3dshapes/C_0603_1608Metric.wrl
@@
   )
   (module Resistor_SMD:R_0603_1608Metric (layer F.Cu)
-    (at 90.424 142.24 180)
+    (at 91.44 141.732 180)
     (descr "Resistor SMD 0603 (1608 Metric), square (rectangular) end terminal, IPC_7351 nominal, (Body size source: http://www.tortai-tech.com/upload/download/2011102023233369053.pdf), generated with kicad-footprint-generator")
     (tags resistor)
@@
   )
   (module Resistor_SMD:R_0603_1608Metric (layer F.Cu)
-    (at 98.044 125.476 180)
+    (at 97.536 130.048 180)
     (descr "Resistor SMD 0603 (1608 Metric), square (rectangular) end terminal, IPC_7351 nominal, (Body size source: http://www.tortai-tech.com/upload/download/2011102023233369053.pdf), generated with kicad-footprint-generator")
     (tags resistor)
@@
   )
   (module Connector_PinSocket_2.54mm:PinSocket_1x02_P2.54mm_Vertical (layer F.Cu)
-    (at 81.788 144.272 90)
+    (at 84.836 144.272 270)
     (descr "Through hole straight socket strip, 1x02, 2.54mm pitch, single row (from Kicad 4.0.7), script generated")
     (tags "Through hole socket strip THT 1x02 2.54mm single row")
@@
       (effects (font (size 1 1) (thickness 0.15)))
     )
-    (pad 1 thru_hole rect (at 0 0 90) (size 1.7 1.7) (drill 1) (layers *.Cu *.Mask)
+    (pad 1 thru_hole rect (at 0 0 270) (size 1.7 1.7) (drill 1) (layers *.Cu *.Mask)
       (net 50 RGB))
-    (pad 2 thru_hole oval (at 0 2.54 90) (size 1.7 1.7) (drill 1) (layers *.Cu *.Mask)
+    (pad 2 thru_hole oval (at 0 2.54 270) (size 1.7 1.7) (drill 1) (layers *.Cu *.Mask)
       (net 54 RGA))
     (model ${KISYS3DMOD}/Connector_PinSocket_2.54mm.3dshapes/PinSocket_1x02_P2.54mm_Vertical.wrl

Commit message: update
Parts:
- moved CF4 30.1 mm to (133.1, 114.8)
- moved RV23G1 23.1 mm to (88.9, 126.0), turned to 180 degrees
- moved U4 23.0 mm to (88.6, 114.3), turned to 90 degrees
- moved J2 22.5 mm to (90.2, 122.4)
- moved RS2 19.9 mm to (103.9, 142.0)
- moved C3 19.4 mm to (133.1, 123.2)
- moved CU11 18.0 mm to (99.3, 130.3), turned to 0 degrees
- moved CF1 17.0 mm to (116.3, 118.9), turned to 90 degrees
- moved R5 16.2 mm to (127.5, 128.8), turned to 270 degrees
- moved CU7 14.8 mm to (83.3, 144.8), turned to 270 degrees
- moved CU5 13.7 mm to (117.3, 123.4)
- moved JRL4 13.4 mm to (81.0, 127.3), turned to 270 degrees
- moved CG2 13.2 mm to (78.2, 145.6)
- moved CG1 12.9 mm to (105.4, 116.3), turned to 180 degrees
- moved RF3 11.7 mm to (111.5, 118.6), turned to 270 degrees
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Connections:
- J1 pad 1: TIA -> V23B
- J1 pad 10: V23C -> PWM1
- J1 pad 11: V23B -> PWM2
- J1 pad 12: V23A -> V12A
- J1 pad 13: RGB -> GNDREF
- J1 pad 14: RGA -> MUXRB
- J1 pad 15: V12C -> MUXRA
- J1 pad 16: V12B -> RGA
- J1 pad 17: V12A -> V23A
- J1 pad 18: PWM2 -> RGB
- J1 pad 19: PWM1 -> VIN4
- J1 pad 2: TIB -> V12C
- J1 pad 20: VIN4 -> VIN2
- J1 pad 21: VIN3 -> MUXVB
- J1 pad 22: VIN2 -> VIN1
- J1 pad 23: VIN1 -> MUXVA
- J1 pad 24: GNDREF -> VIN3
- J1 pad 27: P4 -> P1
- J1 pad 28: P3 -> P2
- J1 pad 29: P2 -> P3
- J1 pad 3: TIC -> MUXGA
- J1 pad 30: P1 -> P4
- J1 pad 4: MUXVA -> TIA
- J1 pad 5: MUXVB -> MUXGB
- J1 pad 6: MUXRA -> V12B
- J1 pad 7: MUXRB -> V23C
- J1 pad 8: MUXGA -> TIC
- J1 pad 9: MUXGB -> TIB
Routing:
- net GND: track 0.00 -> 74.9 mm
- net P1: track 0.00 -> 1.20 mm

Commit message: update
Parts:
- moved CU4 31.0 mm to (94.7, 114.6), turned to 270 degrees
- moved RF7 14.5 mm to (122.9, 127.3), turned to 180 degrees
- moved R6 12.2 mm to (102.9, 136.9)
- moved CU6 5.57 mm to (106.7, 122.4)
- moved R3 4.58 mm to (102.6, 144.0)
- moved RF2 3.06 mm to (109.2, 139.4)
- moved U3 3.05 mm to (100.6, 114.3)
- moved CF2 2.55 mm to (109.2, 143.0)
- moved CU3 2.09 mm to (107.2, 112.0)
- moved U6 2.05 mm to (106.9, 130.8)
- moved CG1 1.80 mm to (107.2, 116.6)
- moved RL1 1.52 mm to (75.7, 126.7), turned to 0 degrees
- moved JRL4 1.27 mm to (82.3, 127.3)
- moved RS2 1.14 mm to (104.4, 141.0)
- moved J2 1.05 mm to (90.4, 121.4)
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Connections:
- J1 pad 13: GNDREF -> MUXRB
- J1 pad 14: MUXRB -> GNDREF
- J1 pad 22: VIN1 -> VIN3
- J1 pad 23: MUXVA -> VIN1
- J1 pad 24: VIN3 -> MUXVA
- J1 pad 4: TIA -> MUXGB
- J1 pad 5: MUXGB -> TIA
Routing:
- net P4: track 0.00 -> 168.9 mm, vias 0 -> 3
- net GND: track 74.9 -> 233.9 mm, vias 0 -> 9
- net VCC: track 0.00 -> 138.2 mm, vias 0 -> 6
- net GNDREF: track 0.00 -> 117.8 mm, vias 0 -> 6
- net P2: track 0.00 -> 87.8 mm, vias 0 -> 5
- net P3: track 0.00 -> 75.2 mm, vias 0 -> 2
- net P1: track 1.20 -> 61.4 mm, vias 0 -> 6
- net TIC: track 0.00 -> 50.4 mm, vias 0 -> 1
- net TIA: track 0.00 -> 48.9 mm, vias 0 -> 4
- net Net-(C1-Pad2): track 0.00 -> 46.7 mm, vias 0 -> 6
- net TIB: track 0.00 -> 46.1 mm, vias 0 -> 1
- net Net-(R34-Pad2): track 0.00 -> 45.5 mm, vias 0 -> 4
- net V23A: track 0.00 -> 42.2 mm, vias 0 -> 5
- net MUXRB: track 0.00 -> 42.0 mm, vias 0 -> 1
- net Net-(R5-Pad2): track 0.00 -> 42.0 mm, vias 0 -> 2
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
Commit message: update
Parts:
- moved R3 2.84 mm to (103.1, 146.8)
Routing:
- net VCC: track 138.2 -> 219.7 mm, vias 6 -> 15
- net GND: track 233.9 -> 295.5 mm, vias 9 -> 17
- net Net-(C84-Pad2): track 0.00 -> 39.0 mm, vias 0 -> 2
- net Net-(R3-Pad2): track 0.00 -> 22.8 mm, vias 0 -> 2
- net RGB: track 16.9 -> 39.2 mm, vias 2 -> 3
- net PWM1: track 36.6 -> 58.3 mm, vias 1 -> 5
- net Net-(RS1-Pad1): track 14.3 -> 35.7 mm, vias 4 -> 6
- net TIA: track 48.9 -> 69.7 mm, vias 4 -> 6
- net Net-(JRV12G1-Pad1): track 5.19 -> 25.3 mm, vias 0 -> 2
- net Net-(RS2-Pad1): track 0.00 -> 19.9 mm
- net GNDREF: track 117.8 -> 136.2 mm, vias 6 -> 10
- net PWM2: track 35.8 -> 53.7 mm, vias 1 -> 5
- net Net-(U3-Pad6): track 0.00 -> 14.0 mm
- net Net-(R6-Pad2): track 0.00 -> 9.89 mm
- net Net-(C5-Pad2): track 14.4 -> 22.9 mm, vias 0 -> 2
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
Commit message: update
Parts:
- J1: value Conn_01x30_Male -> Conn_01x32_Male; footprint Connector_PinHeader_2.54mm:PinHeader_1x30_P2.54mm_Vertical -> Connector_PinHeader_2.54mm:PinHeader_1x32_P2.54mm_Vertical
- moved RF6 6.95 mm to (116.7, 139.4), turned to 90 degrees
- moved CG2 6.33 mm to (83.1, 141.5), turned to 0 degrees
- moved JR4 6.04 mm to (129.5, 138.9)
- moved CF6 5.99 mm to (114.7, 136.1), turned to 270 degrees
- moved JP1 5.85 mm to (71.4, 143.5), turned to 90 degrees
- moved CT4 4.19 mm to (132.1, 135.6)
- moved R3 2.92 mm to (100.2, 146.9)
- moved RS1 2.79 mm to (82.3, 136.4)
- moved RV23G1 1.98 mm to (90.2, 127.5)
- moved CF2 1.52 mm to (109.2, 141.5)
- moved C5 1.45 mm to (112.6, 141.4)
- moved RF1 1.23 mm to (112.0, 113.7)
- moved R34 1.02 mm to (136.7, 143.8)
- moved J1 0.80 mm to (136.9, 104.4)
- moved JRL4 0.77 mm to (82.4, 126.5)
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- renumbered JRV12G1 to JR1, JRG4 to JR4, RV12G1 to RG12
Connections:
- J1 pad 16: RGA -> V23A
- J1 pad 17: V23A -> RG12B
- J1 pad 18: RGB -> RG12A
- J1 pad 19: VIN4 -> RG23B
- J1 pad 20: VIN2 -> RG23A
- J1 pad 21: MUXVB -> VIN4
- J1 pad 22: VIN3 -> VIN2
- J1 pad 23: VIN1 -> MUXVB
- J1 pad 24: MUXVA -> VIN3
- J1 pad 25: GND -> VIN1
- J1 pad 26: VCC -> MUXVA
- J1 pad 27: P1 -> GND
- J1 pad 28: P2 -> VCC
- J1 pad 29: P3 -> P1
- J1 pad 30: P4 -> P2
- J2 pad 1: RGB -> RG23B
- J2 pad 2: RGA -> RG23A
- JR1 pad 1: Net-(JRV12G1-Pad1) -> RG12B
- JR1 pad 2: Net-(JRV12G1-Pad2) -> RG12A
- RG12 pad 1: Net-(JRV12G1-Pad1) -> RG12B
- RG12 pad 2: Net-(JRV12G1-Pad2) -> RG12A
- RV23G1 pad 1: RGB -> RG23B
- RV23G1 pad 2: RGA -> RG23A
- U2 pad 1: Net-(JRV12G1-Pad2) -> RG12A
- U2 pad 8: Net-(JRV12G1-Pad1) -> RG12B
- U4 pad 1: RGA -> RG23A
- U4 pad 8: RGB -> RG23B
Routing:
- net RG12B: track 0.00 -> 57.3 mm, vias 0 -> 5
- net RG12A: track 0.00 -> 41.9 mm, vias 0 -> 7
- net RGB: track 39.2 -> 0.00 mm, vias 3 -> 0
- net RG23B: track 0.00 -> 33.6 mm, vias 0 -> 2
- net RG23A: track 0.00 -> 30.5 mm, vias 0 -> 3
- net RGA: track 28.6 -> 0.00 mm, vias 2 -> 0
- net Net-(JRV12G1-Pad1): track 25.3 -> 0.00 mm, vias 2 -> 0
- net Net-(JRV12G1-Pad2): track 20.3 -> 0.00 mm, vias 4 -> 0
- net TG4: track 41.3 -> 32.9 mm, vias 4 -> 2
- net P1: track 61.4 -> 69.1 mm, vias 6 -> 7
- net TIC: track 50.4 -> 43.2 mm
- net VCC: track 219.7 -> 225.4 mm, vias 15 -> 17
- net P4: track 168.4 -> 163.2 mm
- net V23A: track 42.2 -> 45.8 mm
- net GNDREF: track 136.2 -> 139.1 mm
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Other:
- board size 80.8 x 45.7 mm -> 82.3 x 45.7 mm
- board text added: "4-PROBE CONDUCTIVITY"
- board text added: "ACTINICA & PVOS:"
- board text added: "CURRENT"
- board text added: "GAIN:12"
- board text added: "GAIN:23"
- board text added: "GAIN:i"
- board text added: "GND"
- board text added: "GNDR"
- board text added: "LIMIT:i"
- board text added: "MUXGA"
- board text added: "MUXGB"
- board text added: "MUXRA"
- board text added: "MUXRB"
- board text added: "MUXVA"
- board text added: "MUXVB"
- board text added: "P1"
- board text added: "P2"
- board text added: "P3"
- board text added: "P4"
- board text added: "PWM1"
- board text added: "PWM2"
- board text added: "RG12A"
- board text added: "RG12B"
- board text added: "RG23A"
- board text added: "RG23B"
- board text added: "TIA"
- board text added: "TIB"
- board text added: "TIC"
- board text added: "V12A"
- board text added: "V12B"
- board text added: "V12C"
- board text added: "V23A"
- board text added: "V23B"
- board text added: "V23C"
- board text added: "VCC"
- board text added: "VIN1"
- board text added: "VIN2"
- board text added: "VIN3"
- board text added: "VIN4"
- board text added: "VOLTAGE"
- board text added: "v_0.9"

Commit message: update
Parts:
- removed RV23G1: R, Resistor_SMD:R_0603_1608Metric
- added RG23: R, Resistor_SMD:R_0603_1608Metric, F.Cu at (90.2, 127.5)
- moved CT1 2.48 mm to (136.7, 128.6)
- moved RG2 2.41 mm to (136.7, 132.2)
- moved RG3 2.10 mm to (136.7, 139.6)
- moved CT2 1.97 mm to (136.7, 136.2)
- moved R34 0.71 mm to (136.5, 143.1), turned to 0 degrees
Routing:
- net P4: track 163.2 -> 160.0 mm
- net TG1: track 24.1 -> 21.6 mm
- net Net-(C50-Pad2): track 34.4 -> 32.4 mm
- net Net-(R34-Pad2): track 46.1 -> 47.7 mm

Commit message: update
Parts:
- moved R3 0.70 mm to (99.5, 146.9)
Routing:
- net Net-(C1-Pad2): track 47.3 -> 48.4 mm
- net Net-(R3-Pad2): track 20.2 -> 19.6 mm
Other:
- board text added: "FOUR-PROBE CONDUCTIVITY"
- board text added: "http://pvos.org/four-probe"
- board text removed: "4-PROBE CONDUCTIVITY"
- board text removed: "ACTINICA & PVOS:"
