File: v_0.9/four_probe.kicad_pcb (KiCad board)
At the start: 2 copper layers, 82.3 x 45.7 mm, 79 parts, among them J1 Conn_01x32_Male, J2 RG, J3 CONSMA001-SMD-G, J4 CONSMA001-SMD-G, J5 CONSMA001-SMD-G, J6 CONSMA001-SMD-G, U1 LMC6482, U10 ADG704, U11 tmux1511, U2 AD623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

Commit message: update
Parts:
- moved RG12 1.22 mm to (95.4, 126.3)
- moved RF4 0.89 mm to (136.0, 119.4)
Routing:
- net Net-(CF3-Pad2): track 11.6 -> 10.7 mm
- net V12C: track 28.0 -> 27.4 mm
Other:
- board text added: "GNDREF"
- board text removed: "GNDR"
Changed lines of the file:
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@@
     (thickness 1.6)
     (drawings 63)
-    (tracks 1351)
+    (tracks 1354)
     (zones 0)
     (modules 79)
@@
     (tags resistor)
     (attr smd)
-    (fp_text reference RF1 (at 0 -1.43 90) (layer F.SilkS)
+    (fp_text reference RF1 (at 0 1.397 90) (layer F.SilkS)
       (effects (font (size 1 1) (thickness 0.15)))
     )
@@
   )
   (module Resistor_SMD:R_0603_1608Metric (layer F.Cu)
-    (at 136.906 119.38 90)
+    (at 136.017 119.4435 90)
     (descr "Resistor SMD 0603 (1608 Metric), square (rectangular) end terminal, IPC_7351 nominal, (Body size source: http://www.tortai-tech.com/upload/download/2011102023233369053.pdf), generated with kicad-footprint-generator")
     (tags resistor)
     (attr smd)
-    (fp_text reference RF4 (at 0 -1.43 270) (layer F.SilkS)
+    (fp_text reference RF4 (at 0.0635 1.651 270) (layer F.SilkS)
       (effects (font (size 1 1) (thickness 0.15)))
     )
@@
     (tags resistor)
     (attr smd)
-    (fp_text reference RS3 (at 2.159 0 180) (layer F.SilkS)
+    (fp_text reference RS3 (at -0.0635 -1.4605 270) (layer F.SilkS)
       (effects (font (size 1 1) (thickness 0.15)))
     )
@@
   )
   (module Resistor_SMD:R_0603_1608Metric (layer F.Cu)
-    (at 96.52 125.73 180)
+    (at 95.4405 126.3015 180)
     (descr "Resistor SMD 0603 (1608 Metric), square (rectangular) end terminal, IPC_7351 nominal, (Body size source: http://www.tortai-tech.com/upload/download/2011102023233369053.pdf), generated with kicad-footprint-generator")
     (tags resistor)
@@
     (effects (font (size 0.762 0.762) (thickness 0.127)))
   )
-  (gr_text GNDR (at 104.013 108.458 90) (layer F.SilkS)
+  (gr_text GNDREF (at 104.0765 109.2835 90) (layer F.SilkS)
     (effects (font (size 1.016 1.016) (thickness 0.254)))
   )
@@
   (segment (start 108.4325 139.446) (end 105.09249 136.10599) (width 0.25) (layer F.Cu) (net 11) (status 10))
   (segment (start 108.4325 141.478) (end 108.4325 139.446) (width 0.25) (layer F.Cu) (net 11) (status 30))
-  (segment (start 136.652 119.9135) (end 136.906 120.1675) (width 0.25) (layer F.Cu) (net 12) (status 30))
-  (segment (start 132.08 119.9135) (end 136.652 119.9135) (width 0.25) (layer F.Cu) (net 12) (status 30))
   (via (at 132.08 119.9135) (size 0.8) (drill 0.4) (layers F.Cu B.Cu) (net 12) (status 30))
   (via (at 128.778 121.412) (size 0.8) (drill 0.4) (layers F.Cu B.Cu) (net 12))
@@
   (segment (start 127.508 122.682) (end 127.508 123.604) (width 0.25) (layer F.Cu) (net 12) (status 20))
   (segment (start 128.778 121.412) (end 127.508 122.682) (width 0.25) (layer F.Cu) (net 12))
+  (segment (start 135.6995 119.9135) (end 136.017 120.231) (width 0.25) (layer F.Cu) (net 12))
+  (segment (start 132.08 119.9135) (end 135.6995 119.9135) (width 0.25) (layer F.Cu) (net 12))
   (via (at 131.826 116.84) (size 0.8) (drill 0.4) (layers F.Cu B.Cu) (net 13))
   (segment (start 131.826 118.0845) (end 132.08 118.3385) (width 0.25) (layer F.Cu) (net 13) (status 30))
   (segment (start 131.826 116.84) (end 131.826 118.0845) (width 0.25) (layer F.Cu) (net 13) (status 20))
   (segment (start 132.334 118.5925) (end 132.08 118.3385) (width 0.25) (layer F.Cu) (net 13) (status 30))
-  (segment (start 136.906 118.5925) (end 132.334 118.5925) (width 0.25) (layer F.Cu) (net 13) (status 30))
   (via (at 130.81 122.174) (size 0.8) (drill 0.4) (layers F.Cu B.Cu) (net 13))
   (segment (start 128.778 123.604) (end 129.38 123.604) (width 0.25) (layer F.Cu) (net 13) (status 10))
@@
   (segment (start 134.366 110.998) (end 134.366 104.394) (width 0.25) (layer B.Cu) (net 13) (status 20))
   (segment (start 132.27601 113.08799) (end 134.366 110.998) (width 0.25) (layer B.Cu) (net 13))
+  (segment (start 135.6995 118.3385) (end 136.017 118.656) (width 0.25) (layer F.Cu) (net 13))
+  (segment (start 132.08 118.3385) (end 135.6995 118.3385) (width 0.25) (layer F.Cu) (net 13))
   (segment (start 135.569 114.0205) (end 133.096 114.0205) (width 0.25) (layer F.Cu) (net 14) (status 20))
   (segment (start 136.144 114.0205) (end 135.569 114.0205) (width 0.25) (layer F.Cu) (net 14) (status 10))
@@
   (segment (start 91.948 111.125) (end 91.948 107.696) (width 0.25) (layer F.Cu) (net 66))
   (via (at 94.488 126.492) (size 0.8) (drill 0.4) (layers F.Cu B.Cu) (net 67))
-  (segment (start 95.7325 125.73) (end 95.25 125.73) (width 0.25) (layer F.Cu) (net 67) (status 10))
-  (segment (start 95.25 125.73) (end 94.488 126.492) (width 0.25) (layer F.Cu) (net 67))
-  (via (at 92.456 130.556) (size 0.8) (drill 0.4) (layers F.Cu B.Cu) (net 67))
-  (segment (start 94.488 126.492) (end 92.456 128.524) (width 0.25) (layer B.Cu) (net 67))
-  (segment (start 92.456 128.524) (end 92.456 130.556) (width 0.25) (layer B.Cu) (net 67))
-  (via (at 92.202 132.08) (size 0.8) (drill 0.4) (layers F.Cu B.Cu) (net 67))
-  (segment (start 92.456 130.556) (end 92.456 131.826) (width 0.25) (layer F.Cu) (net 67))
-  (segment (start 92.456 131.826) (end 92.202 132.08) (width 0.25) (layer F.Cu) (net 67))
+  (via (at 91.6305 130.556) (size 0.8) (drill 0.4) (layers F.Cu B.Cu) (net 67))
+  (via (at 91.5035 132.08) (size 0.8) (drill 0.4) (layers F.Cu B.Cu) (net 67))
   (via (at 86.868 134.112) (size 0.8) (drill 0.4) (layers F.Cu B.Cu) (net 67))
-  (segment (start 92.202 132.08) (end 90.17 134.112) (width 0.25) (layer B.Cu) (net 67))
   (segment (start 90.17 134.112) (end 86.868 134.112) (width 0.25) (layer B.Cu) (net 67))
   (segment (start 86.868 135.095) (end 86.708 135.255) (width 0.25) (layer F.Cu) (net 67) (status 30))
   (segment (start 86.868 134.112) (end 86.868 135.095) (width 0.25) (layer F.Cu) (net 67) (status 20))
-  (segment (start 96.266 125.1965) (end 95.7325 125.73) (width 0.25) (layer F.Cu) (net 67) (status 20))
-  (segment (start 96.266 121.158) (end 96.266 125.1965) (width 0.25) (layer F.Cu) (net 67) (status 10))
   (via (at 95.758 111.125) (size 0.8) (drill 0.4) (layers F.Cu B.Cu) (net 67))
   (segment (start 93.726 104.394) (end 95.758 106.426) (width 0.25) (layer F.Cu) (net 67) (status 10))
@@
   (segment (start 95.885 120.777) (end 96.266 121.158) (width 0.25) (layer B.Cu) (net 67) (status 30))
   (segment (start 93.726 120.777) (end 95.885 120.777) (width 0.25) (layer B.Cu) (net 67) (status 20))
-  (segment (start 98.806 124.2315) (end 97.3075 125.73) (width 0.25) (layer F.Cu) (net 68) (status 20))
+  (segment (start 96.266 124.6885) (end 96.266 121.158) (width 0.25) (layer F.Cu) (net 67))
+  (segment (start 94.653 126.3015) (end 96.266 124.6885) (width 0.25) (layer F.Cu) (net 67))
+  (segment (start 90.17 133.4135) (end 91.5035 132.08) (width 0.25) (layer B.Cu) (net 67))
+  (segment (start 90.17 134.112) (end 90.17 133.4135) (width 0.25) (layer B.Cu) (net 67))
+  (segment (start 91.6305 130.556) (end 91.6305 129.3495) (width 0.25) (layer B.Cu) (net 67))
+  (segment (start 94.488 126.492) (end 92.583 128.397) (width 0.25) (layer B.Cu) (net 67))
+  (segment (start 91.6305 129.3495) (end 92.583 128.397) (width 0.25) (layer B.Cu) (net 67))
+  (segment (start 92.583 128.397) (end 92.456 128.524) (width 0.25) (layer B.Cu) (net 67))
+  (segment (start 91.5035 130.683) (end 91.6305 130.556) (width 0.25) (layer F.Cu) (net 67))
+  (segment (start 91.5035 132.08) (end 91.5035 130.683) (width 0.25) (layer F.Cu) (net 67))
   (segment (start 98.806 121.158) (end 98.806 124.2315) (width 0.25) (layer F.Cu) (net 68) (status 10))
   (via (at 97.155 110.617) (size 0.8) (drill 0.4) (layers F.Cu B.Cu) (net 68))
@@
   (segment (start 95.032999 112.739001) (end 91.948 115.824) (width 0.25) (layer B.Cu) (net 68))
   (segment (start 91.948 115.824) (end 91.948 124.968) (width 0.25) (layer B.Cu) (net 68))
-  (segment (start 96.845888 126.191612) (end 97.3075 125.73) (width 0.25) (layer F.Cu) (net 68) (status 20))
-  (segment (start 95.820499 127.217001) (end 96.845888 126.191612) (width 0.25) (layer F.Cu) (net 68))
   (segment (start 91.948 125.533685) (end 93.631316 127.217001) (width 0.25) (layer F.Cu) (net 68))
-  (segment (start 93.631316 127.217001) (end 95.820499 127.217001) (width 0.25) (layer F.Cu) (net 68))
   (segment (start 101.6 125.984) (end 101.200001 126.383999) (width 0.25) (layer B.Cu) (net 68))
   (via (at 101.6 125.984) (size 0.8) (drill 0.4) (layers F.Cu B.Cu) (net 68))
@@
   (segment (start 99.187 121.539) (end 98.806 121.158) (width 0.25) (layer B.Cu) (net 68) (status 30))
   (segment (start 101.473 121.539) (end 99.187 121.539) (width 0.25) (layer B.Cu) (net 68) (status 20))
+  (segment (start 95.312499 127.217001) (end 96.228 126.3015) (width 0.25) (layer F.Cu) (net 68))
+  (segment (start 93.631316 127.217001) (end 95.312499 127.217001) (width 0.25) (layer F.Cu) (net 68))
+  (segment (start 96.228 126.3015) (end 97.3455 126.3015) (width 0.25) (layer F.Cu) (net 68))
+  (segment (start 98.806 124.841) (end 98.806 124.2315) (width 0.25) (layer F.Cu) (net 68))
+  (segment (start 97.3455 126.3015) (end 98.806 124.841) (width 0.25) (layer F.Cu) (net 68))
 )
